File: evaluation-boards/sky13350/sky13350.kicad_pcb (KiCad board)
At the start: 2 copper layers, 42.2 x 32 mm, 19 parts, among them J1 SMA, J2 SMA, J3 SMA, P1 CONN_01X03, P2 CONN_01X03, P3 CONN_01X03, P4 CONN_01X03, P5 CONN_01X03, P6 CONN_01X03, P7 CONN_01X02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

Commit message: finished SKY13350
Parts:
- removed R1, R2, R3, R4: R, gsg-modules:0603
- added C4: 33pF, gsg-modules:0402, F.Cu at (150.0, 99.8)
- added C5: 33pF, gsg-modules:0402, F.Cu at (158.8, 99.8)
- added L1: 15uH, gsg-modules:0603, F.Cu at (148.6, 102.6)
- added L2: 15uH, gsg-modules:0603, F.Cu at (156.2, 102.6)
- added L3: 15uH, gsg-modules:0603, F.Cu at (153.2, 97.8)
- added L4: 15uH, gsg-modules:0603, F.Cu at (152.0, 104.3)
- added L5: 15uH, gsg-modules:0603, F.Cu at (152.8, 107.6)
- C1, C2, C3: value C -> 100nF
Connections:
- P2 pad 2: Net-(P2-Pad2) -> Net-(L5-Pad1)
- U1 pad 3: Net-(P2-Pad2) -> Net-(L4-Pad2)
Routing:
- net Net-(C5-Pad2): track 0.00 -> 24.7 mm
- net Net-(C4-Pad1): track 0.00 -> 24.1 mm
- net Net-(C1-Pad2): track 0.00 -> 8.23 mm
- net Net-(C2-Pad1): track 0.00 -> 8.10 mm
- net Net-(C3-Pad2): track 0.00 -> 7.30 mm
- net Net-(C2-Pad2): track 0.00 -> 6.57 mm
- net Net-(C1-Pad1): track 0.00 -> 6.44 mm
- net Net-(C3-Pad1): track 0.00 -> 6.20 mm
- net Net-(L4-Pad2): track 0.00 -> 4.81 mm
- net Net-(L2-Pad1): track 0.00 -> 3.85 mm
- net Net-(L1-Pad1): track 0.00 -> 3.85 mm
- net GND: track 0.00 -> 3.63 mm, vias 0 -> 3
- net Net-(L5-Pad1): track 0.00 -> 3.60 mm
- net Net-(L3-Pad1): track 0.00 -> 3.02 mm
- added copper zone on C2.Cu, net GND
- added copper zone on C3.Cu, net VCC
Other:
- copper layers 2 -> 4
- net class Default: clearance 0.2 -> 0.1524; trace_width 0.25 -> 0.3048; via_dia 0.6 -> 1.016; via_drill 0.4 -> 0.508
- rule trace_clearance: 0.2 -> 0.1524
- board text added: "GND"
- board text added: "J1 OUT1"
- board text added: "J2 OUT2"
- board text added: "J3 IN"
- board text added: "P3 VCTL1"
- board text added: "P4 VCTL2"
- board text added: "SKY13350 5 March 2016"
- board text added: "VCC"
