File: evaluation-boards/sky13351/sky13351.kicad_pcb (KiCad board)
At the start: 4 copper layers, 42.2 x 32 mm, 22 parts, among them J1 SMA, J2 SMA, J3 SMA, P1 CONN_01X03, P2 CONN_01X03, P3 CONN_01X03, P4 CONN_01X03, P5 CONN_01X03, P6 CONN_01X03, P7 CONN_01X02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

Commit message: SKY13351 evaluation board
Parts:
- U1: value SKY13350 -> SKY13351; footprint gsg-modules:SKY13350-385LF -> gsg-modules:SKY13351-378LF
- turned U1 to 90 degrees
Connections:
- U1 pad 1: Net-(C4-Pad1) -> Net-(C1-Pad1)
- U1 pad 2: Net-(C1-Pad1) -> Net-(L4-Pad2)
- U1 pad 3: Net-(L4-Pad2) -> Net-(C2-Pad2)
- U1 pad 4: Net-(C2-Pad2) -> Net-(C5-Pad2)
- U1 pad 5: Net-(C5-Pad2) -> Net-(C3-Pad2)
- U1 pad 6: Net-(C3-Pad2) -> Net-(C4-Pad1)
Other:
- rule trace_min: 0.2 -> 0.1778
- board text added: "SKY13351 5 March 2016"
- board text removed: "SKY13350 5 March 2016"
