File: evaluation-boards/CC-test/CC-test.sch (KiCad schematic (older format))
At the start: 27 parts, among them J1 Conn_02x06_Top_Bottom, J2 Conn_01x02, J3 Conn_01x02, J4 Conn_01x02, J5 Conn_01x02, J6 USB_C_Receptacle_USB2.0, J7 Conn_01x02, J8 Conn_01x02, U1 MIC5504-1.8YM5, U2 74AUP2G126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

Commit message: CC-test: change U2 and U3 to 74AUP2G126RA3-7
Parts:
- U2, U3: footprint CC-test:XSON-8_1.95x1mm_P0.5mm -> CC-test:X2-DFN1210-8_1.2x1mm_P0.3mm; Manufacturer (none) -> Diodes, Inc.; Part Number (none) -> 74AUP2G126RA3-7
