File: evaluation-boards/pmos-or/pmos-or.kicad_pcb (KiCad board)
At the start: 2 copper layers, 74 x 59 mm, 46 parts, among them J1 IN1, J10 GND, J2 IN2, J3 OUT, J4 USB_C_Receptacle_USB2.0, J5 USB_C_Receptacle_USB2.0, J6 USB_A, J7 IN1, J8 OUT, J9 IN2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

Commit message: pmos-or: add part selections
Other:
- board text added: "pmos-or 2023-01-24"
- board text removed: "pmos-or 2023-01-23"
Changed lines of the file:
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@@
     (descr "SOT, 3 Pin (https://www.jedec.org/sites/default/files/docs/Mo-178D.PDF inferred 3-pin variant), generated with kicad-footprint-generator ipc_gullwing_generator.py")
     (tags "SOT TO_SOT_SMD")
+    (property "Manufacturer" "Panjit")
+    (property "Part Number" "PJA3441_R1_00001")
     (property "Sheetfile" "pmos-or.kicad_sch")
     (property "Sheetname" "")
@@
     (at 133 85 -90)
     (property "DNP" "DNP")
+    (property "Manufacturer" "Nexperia")
+    (property "Part Number" "PMEG3050BEP,115")
     (property "Sheetfile" "pmos-or.kicad_sch")
     (property "Sheetname" "")
@@
     (descr "SOT, 3 Pin (https://www.jedec.org/sites/default/files/docs/Mo-178D.PDF inferred 3-pin variant), generated with kicad-footprint-generator ipc_gullwing_generator.py")
     (tags "SOT TO_SOT_SMD")
+    (property "Manufacturer" "Panjit")
+    (property "Part Number" "PJA3441_R1_00001")
     (property "Sheetfile" "pmos-or.kicad_sch")
     (property "Sheetname" "")
@@
     (descr "USB Type-C receptacle for USB 2.0 and PD, http://www.krhro.com/uploads/soft/180320/1-1P320120243.pdf")
     (tags "USB_C female connector receptacle type-c usb-2.0 usb pd")
+    (property "Manufacturer" "XKB")
+    (property "Part Number" "U262-161N-4BVC11")
     (property "Sheetfile" "pmos-or.kicad_sch")
     (property "Sheetname" "")
@@
     (descr "SOT-363, SC-70-6")
     (tags "SOT-363 SC-70-6")
+    (property "Manufacturer" "Diodes Inc.")
+    (property "Part Number" "BCM857BS-7-F")
     (property "Sheetfile" "pmos-or.kicad_sch")
     (property "Sheetname" "")
@@
     (at 167 85 -90)
     (property "DNP" "DNP")
+    (property "Manufacturer" "Nexperia")
+    (property "Part Number" "PMEG3050BEP,115")
     (property "Sheetfile" "pmos-or.kicad_sch")
     (property "Sheetname" "")
@@
     (descr "SOT-363, SC-70-6")
     (tags "SOT-363 SC-70-6")
+    (property "Manufacturer" "Yangzhou Yangjie")
+    (property "Part Number" "2N7002DW")
     (property "Sheetfile" "pmos-or.kicad_sch")
     (property "Sheetname" "")
@@
     (descr "SOT-363, SC-70-6")
     (tags "SOT-363 SC-70-6")
+    (property "Manufacturer" "Yangzhou Yangjie")
+    (property "Part Number" "BSS84DW")
     (property "Sheetfile" "pmos-or.kicad_sch")
     (property "Sheetname" "")
@@
     (descr "SOT, 3 Pin (https://www.jedec.org/sites/default/files/docs/Mo-178D.PDF inferred 3-pin variant), generated with kicad-footprint-generator ipc_gullwing_generator.py")
     (tags "SOT TO_SOT_SMD")
+    (property "Manufacturer" "Panjit")
+    (property "Part Number" "PJA3441_R1_00001")
     (property "Sheetfile" "pmos-or.kicad_sch")
     (property "Sheetname" "")
@@
     (property "Sheetname" "")
     (attr smd)
-    (fp_text reference "D3" (at 0 -0.9 -90) (layer "F.SilkS")
-      (effects (font (size 0.5 0.5) (thickness 0.1)))
+    (fp_text reference "D3" (at -1.6 0) (layer "F.SilkS")
+      (effects (font (size 1 1) (thickness 0.15)))
     )
     (fp_text value "4.7±2%" (at 0 1.6 -90 unlocked) (layer "F.Fab")
@@
     (fp_rect (start -0.65 -0.45) (end 0.65 0.45) (layer "F.SilkS") (width 0.1) (fill none))
     (fp_rect (start -0.65 -0.45) (end 0.65 0.45) (layer "F.CrtYd") (width 0.05) (fill none))
+    (fp_line (start 0.15 -0.15) (end 0.15 0.15) (layer "F.Fab") (width 0.1))
+    (fp_line (start -0.2 -0.15) (end -0.2 0.15) (layer "F.Fab") (width 0.1))
     (fp_line (start -0.1 0) (end 0.15 -0.15) (layer "F.Fab") (width 0.1))
-    (fp_line (start -0.2 -0.15) (end -0.2 0.15) (layer "F.Fab") (width 0.1))
-    (fp_line (start 0.15 -0.15) (end 0.15 0.15) (layer "F.Fab") (width 0.1))
     (fp_line (start 0.15 0.15) (end -0.1 0) (layer "F.Fab") (width 0.1))
     (fp_rect (start -0.5 -0.3) (end 0.5 0.3) (layer "F.Fab") (width 0.1) (fill none))
@@
     (descr "USB Type-C receptacle for USB 2.0 and PD, http://www.krhro.com/uploads/soft/180320/1-1P320120243.pdf")
     (tags "USB_C female connector receptacle type-c usb-2.0 usb pd")
+    (property "Manufacturer" "XKB")
+    (property "Part Number" "U262-161N-4BVC11")
     (property "Sheetfile" "pmos-or.kicad_sch")
     (property "Sheetname" "")
@@
     (descr "USB A connector http://www.kycon.com/Pub_Eng_Draw/KUSBXHT-SB-AS1N-B30-NF.pdf")
     (tags "USB_A female connector receptacle type-a usb-2.0")
+    (property "Manufacturer" "Jing Extension of the Electronic Co.")
+    (property "Part Number" "C42411")
     (property "Sheetfile" "pmos-or.kicad_sch")
     (property "Sheetname" "")
@@
     (effects (font (size 2 2) (thickness 0.3)))
   )
-  (gr_text "pmos-or\n2023-01-23" (at 149.5 117.8) (layer "F.SilkS")
+  (gr_text "pmos-or\n2023-01-24" (at 149.5 117.8) (layer "F.SilkS")
     (effects (font (size 1 1) (thickness 0.15)))
   )
