File: evaluation-boards/vbus-switch/vbus-switch.kicad_pcb (KiCad board)
At the start: 4 copper layers, 74 x 59 mm, 83 parts, among them J1 BANANA, J10 01x02, J11 Conn_02x06_Top_Bottom, J2 BANANA, J3 BANANA, J4 USB_C, J5 USB_C, J6 USB_A, J7 01x02, J8 01x02, J9 01x02, Q1 PMOS, Q2 PMOS, Q3 PMOS, Q4 PMOS, Q5 2PMOS, Q6 2NMOS, Q7 2NMOS, U1 PAC195X-1-WLCSP, U2 FUSB302BMPX

Commit message: update vbus-switch
Parts:
- added C11: 2.2uF, Capacitor_SMD:C_0603_1608Metric, F.Cu at (147.9, 130.2)
- added C12: 1uF, Capacitor_SMD:C_0603_1608Metric, F.Cu at (149.9, 122.7)
- added C13: 390pF, Capacitor_SMD:C_0402_1005Metric, F.Cu at (130.3, 136.9)
- added C14: 390pF, Capacitor_SMD:C_0402_1005Metric, F.Cu at (127.3, 136.9)
- added C15: 390pF, Capacitor_SMD:C_0402_1005Metric, F.Cu at (124.2, 90.3)
- added C16: 390pF, Capacitor_SMD:C_0402_1005Metric, F.Cu at (124.2, 86.3)
- added D3: D, Diode_SMD:D_SOD-123F, F.Cu at (142.0, 115.0)
- added D4: 6.2±2%, eval:DFN1006-2, F.Cu at (145.5, 115.5)
- added D5: D, Diode_SMD:D_SOD-123F, F.Cu at (142.0, 120.0)
- added D6: 18±2%, eval:DFN1006-2, F.Cu at (137.0, 117.0)
- added D7: 4.7±2%, eval:DFN1006-2, F.Cu at (134.2, 124.0)
- added J12: 01x02, Connector_PinHeader_2.54mm:PinHeader_1x02_P2.54mm_Vertical, F.Cu at (142.0, 128.0)
- added J13: BANANA, Connector:Banana_Jack_2Pin, F.Cu at (172.0, 141.0)
- added J14: 01x02, Connector_PinHeader_2.54mm:PinHeader_1x02_P2.54mm_Vertical, F.Cu at (147.0, 119.8)
- added J15: 01x02, Connector_PinHeader_2.54mm:PinHeader_1x02_P2.54mm_Vertical, F.Cu at (156.0, 130.8)
- added J16: 01x02, Connector_PinHeader_2.54mm:PinHeader_1x02_P2.54mm_Vertical, F.Cu at (156.0, 118.0)
- added J17: USB_C, eval:USB_C_Receptacle_HRO_TYPE-C-31-M-12, F.Cu at (129.0, 145.1)
- added Q10: 2NPN, Package_TO_SOT_SMD:SOT-363_SC-70-6, F.Cu at (168.1, 101.4)
- added Q11: PMOS, Package_TO_SOT_SMD:SOT-23-3, F.Cu at (163.7, 99.4)
- added Q12: PMOS, Package_TO_SOT_SMD:SOT-23-3, F.Cu at (163.7, 103.5)
- added Q8: PMOS, Package_TO_SOT_SMD:SOT-23-3, F.Cu at (145.7, 99.4)
- added Q9: PMOS, Package_TO_SOT_SMD:SOT-23-3, F.Cu at (150.6, 99.4)
- added R37: 33k, Resistor_SMD:R_0402_1005Metric, F.Cu at (157.6, 99.3)
- added R38: 33k, Resistor_SMD:R_0402_1005Metric, F.Cu at (154.7, 104.0)
- added R39: 2.2k, Resistor_SMD:R_0402_1005Metric, F.Cu at (152.8, 93.4)
- added R40: 2.2k, Resistor_SMD:R_0402_1005Metric, F.Cu at (159.9, 90.5)
- added R41: 18.7k±1%, Resistor_SMD:R_0402_1005Metric, F.Cu at (163.6, 113.1)
- added R42: 2.2k, Resistor_SMD:R_0402_1005Metric, F.Cu at (168.1, 95.6)
- added R43: 33k, Resistor_SMD:R_0402_1005Metric, F.Cu at (168.7, 98.9)
- added R44: 33k, Resistor_SMD:R_0402_1005Metric, F.Cu at (166.0, 105.9)
- added R45: 33k, Resistor_SMD:R_0402_1005Metric, F.Cu at (163.7, 96.7)
- added R46: 0.02±1%, eval:R_0603_1608Metric_Current_Sense, F.Cu at (165.7, 114.4)
- added R47: 0, Resistor_SMD:R_0402_1005Metric, F.Cu at (133.8, 138.1)
- added R48: 58.3k±1%, Resistor_SMD:R_0402_1005Metric, F.Cu at (151.3, 131.1)
- added R49: R, Resistor_SMD:R_0402_1005Metric, F.Cu at (131.9, 93.7)
- added R50: R, Resistor_SMD:R_0402_1005Metric, F.Cu at (165.2, 118.1)
- added R51: 18.7k±1%, Resistor_SMD:R_0402_1005Metric, F.Cu at (152.5, 131.1)
- added R52: 5.1k, Resistor_SMD:R_0402_1005Metric, F.Cu at (130.3, 135.7)
- added R53: 5.1k, Resistor_SMD:R_0402_1005Metric, F.Cu at (127.3, 135.7)
- added R54: R, Resistor_SMD:R_0402_1005Metric, F.Cu at (131.1, 132.3)
- added TP16: TestPoint, TestPoint:TestPoint_Pad_D1.5mm, F.Cu at (130.6, 128.2)
- added U3: AP7361EA-33, Package_DFN_QFN:DFN-8-1EP_3x3mm_P0.65mm_EP1.55x2.4mm, F.Cu at (150.8, 127.0)
- C1: footprint Capacitor_SMD:C_0805_2012Metric -> Capacitor_SMD:C_0402_1005Metric
- D1: value 5.6±2% -> 4.7±2%
- D2: value 4.7±2% -> 18±2%
- Q1: value PMOS -> 2NPN; footprint Package_TO_SOT_SMD:SOT-23-3 -> Package_TO_SOT_SMD:SOT-363_SC-70-6
- Q2: value PMOS -> 2PNP; footprint Package_TO_SOT_SMD:SOT-23-3 -> Package_TO_SOT_SMD:SOT-363_SC-70-6
- Q5: value 2PMOS -> PMOS; footprint Package_TO_SOT_SMD:SOT-363_SC-70-6 -> Package_TO_SOT_SMD:SOT-23-3
- Q6: value 2NMOS -> PMOS; footprint Package_TO_SOT_SMD:SOT-363_SC-70-6 -> Package_TO_SOT_SMD:SOT-23-3
- Q7: value 2NMOS -> 2NPN
- R1, R2, R21: value 20k -> 18.7k±1%
- R13: value 0 -> 2.2k
- R14: value 1k -> 33k
- R15: value 1k -> 18.7k±1%
- R16: value 20k -> R
- R17, R22, R29, R30: value 10k -> 18.7k±1%
- R18, R33: value 10k -> 33k
- R20: value 10k -> 2.2k
- R3, R4: value 0.02±1% -> 18.7k±1%; footprint eval:R_0603_1608Metric_Current_Sense -> Resistor_SMD:R_0402_1005Metric
- R31: value 20k -> 0.02±1%; footprint Resistor_SMD:R_0402_1005Metric -> eval:R_0603_1608Metric_Current_Sense
- R32: value 10k -> 0.02±1%; footprint Resistor_SMD:R_0402_1005Metric -> eval:R_0603_1608Metric_Current_Sense
- R35: value 0.02±1% -> 33k; footprint eval:R_0603_1608Metric_Current_Sense -> Resistor_SMD:R_0402_1005Metric
- moved R20 51.3 mm to (128.5, 125.1), turned to -90 degrees
- moved R30 46.3 mm to (132.0, 125.0), turned to 180 degrees
- moved TP5 44.5 mm to (127.1, 81.7), turned to 180 degrees
- moved C1 43.4 mm to (146.9, 125.8)
- moved R32 40.5 mm to (137.6, 127.2), turned to -90 degrees
- moved C4 40.2 mm to (133.7, 132.3), turned to 0 degrees
- moved R21 39.3 mm to (129.8, 122.8)
- moved R13 39.2 mm to (127.1, 117.3), turned to 90 degrees
- moved R1 38.3 mm to (131.4, 111.5), turned to 180 degrees
- moved TP9 37.3 mm to (133.8, 80.6), turned to 180 degrees
- moved R29 36.7 mm to (135.2, 121.5)
- moved J4 36.3 mm to (115.9, 88.0), turned to -90 degrees
- moved R24 36.2 mm to (130.2, 84.5), turned to 180 degrees
- moved TP4 35.5 mm to (134.1, 127.3), turned to 180 degrees
- moved R16 35.2 mm to (146.9, 128.2), turned to 0 degrees
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Connections:
- net VBUS_A renamed TARGET_A_VBUS_CONN
- C1 pad 1: VBUS_CAP -> +5V
- C4 pad 1: /VBUS -> AUX_VBUS_CONN
- C5 pad 1: VBUS_C -> TARGET_C_VBUS_CONN
- C7 pad 1: +5V -> CONTROL_VBUS_CONN
- D1 pad 2: GND -> Net-(D1-Pad2)
- D2 pad 1: /VBUS -> CONTROL_VBUS
- J1 pad 2: +5V -> CONTROL_VBUS_CONN
- J11 pad 7: VBUS_C_EN -> ~{TARGET_C_VBUS_EN}
- J11 pad 8: VBUS_A_EN -> AUX_VBUS_EN
- J11 pad 9: 5V_OUT_EN -> CONTROL_VBUS_EN
- J2 pad 2: VBUS_C -> TARGET_C_VBUS_CONN
- J4 pad A4: +5V -> CONTROL_VBUS_CONN
- J4 pad A9: +5V -> CONTROL_VBUS_CONN
- J4 pad B4: +5V -> CONTROL_VBUS_CONN
- J4 pad B9: +5V -> CONTROL_VBUS_CONN
- J5 pad A4: VBUS_C -> TARGET_C_VBUS_CONN
- J5 pad A9: VBUS_C -> TARGET_C_VBUS_CONN
- J5 pad B4: VBUS_C -> TARGET_C_VBUS_CONN
- J5 pad B9: VBUS_C -> TARGET_C_VBUS_CONN
- J7 pad 1: +5V -> CONTROL_VBUS_CONN
- J7 pad 2: +5V -> CONTROL_VBUS_CONN
- J9 pad 1: VBUS_C -> TARGET_C_VBUS_CONN
- J9 pad 2: VBUS_C -> TARGET_C_VBUS_CONN
- Q1 pad 1: Net-(Q1-Pad1) -> GND
- Q1 pad 2: /VBUS -> Net-(Q1-Pad2)
- Q2 pad 1: Net-(Q2-Pad1) -> CONTROL_VBUS
- Q2 pad 2: /VBUS -> Net-(D1-Pad1)
- Q2 pad 3: Net-(Q2-Pad3) -> Net-(D6-Pad2)
- Q3 pad 1: Net-(Q3-Pad1) -> Net-(D2-Pad2)
- Q3 pad 2: /VBUS -> Net-(D3-Pad2)
- Q3 pad 3: Net-(Q3-Pad3) -> CONTROL_VBUS
- Q4 pad 1: Net-(Q3-Pad1) -> Net-(D6-Pad2)
- Q4 pad 2: /VBUS -> Net-(D5-Pad2)
- Q4 pad 3: Net-(Q4-Pad3) -> AUX_VBUS
- Q5 pad 1: /VBUS -> Net-(Q5-Pad1)
- Q5 pad 3: Net-(Q1-Pad1) -> CONTROL_VBUS
- Q6 pad 1: GND -> Net-(Q6-Pad1)
- Q6 pad 2: VBUS_A_EN -> Net-(Q6-Pad2)
- Q6 pad 3: Net-(Q6-Pad3) -> AUX_VBUS
- Q7 pad 2: Net-(D2-Pad2) -> Net-(Q7-Pad2)
- Q7 pad 3: Net-(Q7-Pad3) -> Net-(Q6-Pad1)
- Q7 pad 6: Net-(Q7-Pad5) -> Net-(Q5-Pad1)
- R1 pad 1: /VBUS -> CONTROL_VBUS
- R1 pad 2: Net-(Q2-Pad1) -> Net-(D1-Pad1)
- R13 pad 1: VBUS_CAP -> Net-(Q1-Pad2)
- R13 pad 2: Net-(D1-Pad1) -> ~{CONTROL_VBUS_IN_EN}
- R14 pad 1: Net-(Q7-Pad5) -> CONTROL_VBUS
- R14 pad 2: 5V_OUT_EN -> Net-(D2-Pad2)
- R16 pad 1: /VBUS -> +5V
- R16 pad 2: Net-(Q3-Pad1) -> GND
- R17 pad 1: Net-(Q7-Pad5) -> Net-(D6-Pad2)
- R18 pad 1: Net-(Q3-Pad1) -> AUX_VBUS
- R18 pad 2: Net-(Q7-Pad3) -> Net-(D6-Pad2)
- R2 pad 1: /VBUS -> Net-(D1-Pad2)
- R2 pad 2: Net-(Q1-Pad1) -> GND
- R20 pad 1: VBUS_A_EN -> Net-(Q1-Pad5)
- R20 pad 2: GND -> ~{AUX_VBUS_IN_EN}
- R21 pad 1: Net-(Q5-Pad2) -> Net-(Q1-Pad5)
- R21 pad 2: /VBUS -> GND
- R22 pad 1: Net-(Q5-Pad2) -> Net-(D7-Pad1)
- R22 pad 2: Net-(Q6-Pad6) -> Net-(Q1-Pad3)
- R29 pad 1: Net-(Q2-Pad1) -> AUX_VBUS
- R29 pad 2: GND -> Net-(D7-Pad1)
- R3 pad 1: VBUS_CAP -> Net-(D1-Pad1)
- R3 pad 2: CAP_SENSE+ -> Net-(Q1-Pad6)
- R30 pad 1: VBUS_C_EN -> Net-(D7-Pad2)
- R31 pad 1: Net-(Q5-Pad5) -> CONTROL_VBUS_CONN
- R31 pad 2: /VBUS -> CONTROL_SENSE+
- R32 pad 1: Net-(Q5-Pad5) -> AUX_VBUS
- R32 pad 2: Net-(Q6-Pad3) -> AUX_SENSE-
- R33 pad 1: Net-(Q1-Pad1) -> Net-(Q5-Pad2)
- R33 pad 2: GND -> Net-(Q5-Pad1)
- R34 pad 1: Net-(Q2-Pad3) -> TARGET_A_VBUS
- R34 pad 2: VBUS_A_SENSE- -> TARGET_A_SENSE-
- R34 pad 3: VBUS_A_SENSE+ -> TARGET_A_SENSE+
- R35 pad 1: Net-(Q1-Pad3) -> Net-(Q6-Pad2)
- R35 pad 2: VBUS_C_SENSE- -> Net-(Q6-Pad1)
- R4 pad 1: Net-(Q3-Pad3) -> Net-(Q1-Pad2)
- R4 pad 2: 5V_SENSE- -> GND
- TP1 pad 1: VBUS_CAP -> Net-(D1-Pad1)
- TP10 pad 1: Net-(Q2-Pad1) -> Net-(Q5-Pad1)
- TP11 pad 1: Net-(Q5-Pad5) -> Net-(Q6-Pad1)
- TP12 pad 1: Net-(Q1-Pad1) -> TARGET_A_VBUS
- TP13 pad 1: Net-(D2-Pad2) -> Net-(Q10-Pad5)
- TP14 pad 1: Net-(Q7-Pad5) -> Net-(Q10-Pad3)
- TP15 pad 1: /VBUS -> ~{CONTROL_VBUS_IN_EN}
- TP2 pad 1: Net-(D1-Pad1) -> Net-(D2-Pad2)
- TP3 pad 1: Net-(Q3-Pad1) -> Net-(D6-Pad2)
- TP4 pad 1: Net-(Q5-Pad2) -> Net-(D7-Pad1)
- U1 pad A1: VBUS_A_SENSE+ -> CONTROL_SENSE+
- U1 pad A2: VBUS_C_SENSE- -> AUX_SENSE-
- U1 pad A3: VBUS_C_SENSE+ -> AUX_SENSE+
- U1 pad B1: VBUS_A_SENSE- -> CONTROL_SENSE-
- U1 pad C1: CAP_SENSE- -> TARGET_C_SENSE-
- U1 pad D1: CAP_SENSE+ -> TARGET_C_SENSE+
- U1 pad D2: 5V_SENSE- -> TARGET_A_SENSE-
- U1 pad D3: 5V_SENSE+ -> TARGET_A_SENSE+
- U2 pad 2: VBUS_C -> Net-(U2-Pad2)
Routing:
- net 5V_OUT_EN: track 70.8 -> 0.00 mm, vias 2 -> 0
- net /SCL: track 59.6 -> 127.8 mm, vias 1 -> 3
- net VBUS_C: track 56.1 -> 0.00 mm
- net AUX_SENSE+: track 0.00 -> 55.1 mm, vias 0 -> 2
- net AUX_SENSE-: track 0.00 -> 54.3 mm, vias 0 -> 2
- net TARGET_A_VBUS: track 0.00 -> 50.8 mm
- net CONTROL_VBUS_CONN: track 0.00 -> 48.0 mm
- net TARGET_C_SENSE+: track 0.00 -> 47.5 mm, vias 0 -> 2
- net TARGET_C_SENSE-: track 0.00 -> 47.5 mm, vias 0 -> 2
- net /SDA: track 69.8 -> 117.0 mm, vias 1 -> 3
- net AUX_VBUS_CONN: track 0.00 -> 46.7 mm
- net CONTROL_VBUS_EN: track 0.00 -> 43.0 mm, vias 0 -> 2
- net /VBUS: track 41.2 -> 0.00 mm
- net TARGET_C_VBUS_CONN: track 0.00 -> 40.9 mm
- net AUX_VBUS: track 0.00 -> 36.0 mm
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- added copper zone on F.Cu, net Net-(J17-PadS1)
Other:
- board size 74 x 59 mm -> 74 x 85 mm
- board text added: "Aux"
- board text added: "Control"
- board text added: "Target A"
- board text added: "Target C"
- board text added: "vbus-switch ${ISSUE_DATE}"
- board text removed: "+5V"
- board text removed: "VBUS_A"
- board text removed: "VBUS_C"
- board text removed: "vbus-switch 2023-01-24"

Commit message: vbus-switch: update resistor selection
Parts:
- R14, R18: value 33k -> 820k
- R15, R17, R22, R3: value 18.7k±1% -> 33k
- R2, R30: value 18.7k±1% -> 22k±1%
- R21, R4: value 18.7k±1% -> 10k
- R37, R38, R43: value 33k -> 10k
- R41: value 18.7k±1% -> 20k
Connections:
- net Net-(C11-Pad1) renamed /3V3OUT
