File: evaluation-boards/vbus-switch/vbus-switch.kicad_sch (KiCad schematic)
At the start: 125 parts, among them J1 BANANA, J10 01x02, J11 Conn_02x06_Top_Bottom, J12 01x02, J13 BANANA, J14 01x02, J15 01x02, J16 01x02, J17 USB_C, J2 BANANA, J3 BANANA, J4 USB_C, J5 USB_C, J6 USB_A, J7 01x02, J8 01x02, J9 01x02, Q1 2NPN, Q10 2NPN, Q11 PMOS, Q12 PMOS, Q2 2PNP, Q3 PMOS, Q4 PMOS, Q5 PMOS, Q6 PMOS, Q7 2NPN, Q8 PMOS, Q9 PMOS, U1 PAC195X-1-WLCSP, U2 FUSB302BMPX, U3 AP7361EA-33

Commit message: vbus-switch: update resistor selection
Parts:
- R14, R18: value 33k -> 820k
- R15, R17, R22, R3: value 18.7k±1% -> 33k
- R2, R30: value 18.7k±1% -> 22k±1%
- R21, R4: value 18.7k±1% -> 10k
- R37, R38, R43: value 33k -> 10k
- R41: value 18.7k±1% -> 20k
Connections:
- net 3V3OUT: now reaches C11.1, J15.1 (Pin_1), J15.2 (Pin_2), R48.1, U3.1 (OUT)
Other:
- note added: "+5V required: 3.8 to 6.0 V absolute max: 6.5 V"
- note added: "AUX_VBUS expected: 4.4 to 21 V absolute max: 40 V"
- note added: "CONTROL_VBUS expected: 4.4 to 5.5 V absolute max: 40 V"
- note added: "FUSB302B VBUS input recommended max: 21 V absolute max: 28 V protected from higher voltage by resistor"
- note added: "TARGET_A_VBUS expected: 4.4 to 21 V absolute max: 40 V"
- note added: "TARGET_C_VBUS expected: 4.4 to 21 V absolute max: 40 V"
- note removed: "recommended max: 20 V absolute max: 28 V"
Changed lines of the file:
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@@
     (stroke (width 0) (type default) (color 0 0 0 0))
   )
-  (text "recommended max: 20 V\nabsolute max: 28 V" (at 352.425 163.195 0)
+  (text "CONTROL_VBUS\nexpected: 4.4 to 5.5 V\nabsolute max: 40 V"
+    (at 36.195 31.75 0)
+    (effects (font (size 1.27 1.27)) (justify left bottom))
+  )
+  (text "+5V\nrequired: 3.8 to 6.0 V\nabsolute max: 6.5 V" (at 142.24 108.585 0)
+    (effects (font (size 1.27 1.27)) (justify left bottom))
+  )
+  (text "AUX_VBUS\nexpected: 4.4 to 21 V\nabsolute max: 40 V" (at 192.405 32.385 0)
+    (effects (font (size 1.27 1.27)) (justify left bottom))
+  )
+  (text "FUSB302B VBUS input\nrecommended max: 21 V\nabsolute max: 28 V\nprotected from higher voltage by resistor"
+    (at 288.29 178.435 0)
+    (effects (font (size 1.27 1.27)) (justify left bottom))
+  )
+  (text "TARGET_C_VBUS\nexpected: 4.4 to 21 V\nabsolute max: 40 V"
+    (at 381.2453 89.738 0)
+    (effects (font (size 1.27 1.27)) (justify left bottom))
+  )
+  (text "TARGET_A_VBUS\nexpected: 4.4 to 21 V\nabsolute max: 40 V"
+    (at 381.635 38.1 0)
     (effects (font (size 1.27 1.27)) (justify left bottom))
   )
@@
     (effects (font (size 1.27 1.27)) (justify left bottom))
   )
+  (label "3V3OUT" (at 109.22 116.205 0)
+    (effects (font (size 1.27 1.27)) (justify left bottom))
+  )
   (label "VCONN" (at 281.94 199.39 90)
     (effects (font (size 1.27 1.27)) (justify left bottom))
@@
       (effects (font (size 1.27 1.27)) (justify left))
     )
-    (property "Value" "18.7k±1%" (id 1) (at 77.978 77.9022 0)
+    (property "Value" "10k" (id 1) (at 77.978 77.9022 0)
       (effects (font (size 1.27 1.27)) (justify left))
     )
@@
       (effects (font (size 1.27 1.27)) (justify left))
     )
-    (property "Value" "33k" (id 1) (at 297.053 111.5572 0)
+    (property "Value" "10k" (id 1) (at 297.053 111.5572 0)
       (effects (font (size 1.27 1.27)) (justify left))
     )
@@
       (effects (font (size 1.27 1.27)) (justify left))
     )
-    (property "Value" "18.7k±1%" (id 1) (at 58.928 77.9022 0)
+    (property "Value" "22k±1%" (id 1) (at 58.928 77.9022 0)
       (effects (font (size 1.27 1.27)) (justify left))
     )
@@
       (effects (font (size 1.27 1.27)) (justify left))
     )
-    (property "Value" "18.7k±1%" (id 1) (at 69.088 59.4872 0)
+    (property "Value" "33k" (id 1) (at 69.088 59.4872 0)
       (effects (font (size 1.27 1.27)) (justify left))
     )
@@
       (effects (font (size 1.27 1.27)) (justify left))
     )
-    (property "Value" "33k" (id 1) (at 160.147 48.0572 0)
+    (property "Value" "820k" (id 1) (at 160.147 48.0572 0)
       (effects (font (size 1.27 1.27)) (justify left))
     )
@@
       (effects (font (size 1.27 1.27)) (justify left))
     )
-    (property "Value" "33k" (id 1) (at 325.247 117.9072 0)
+    (property "Value" "10k" (id 1) (at 325.247 117.9072 0)
       (effects (font (size 1.27 1.27)) (justify left))
     )
@@
       (effects (font (size 1.27 1.27)) (justify left))
     )
-    (property "Value" "18.7k±1%" (id 1) (at 105.918 62.0272 0)
+    (property "Value" "33k" (id 1) (at 105.918 62.0272 0)
       (effects (font (size 1.27 1.27)) (justify left))
     )
@@
       (effects (font (size 1.27 1.27)) (justify left))
     )
-    (property "Value" "18.7k±1%" (id 1) (at 188.087 77.9022 0)
+    (property "Value" "22k±1%" (id 1) (at 188.087 77.9022 0)
       (effects (font (size 1.27 1.27)) (justify left))
     )
@@
       (effects (font (size 1.27 1.27)) (justify left))
     )
-    (property "Value" "18.7k±1%" (id 1) (at 141.097 62.0272 0)
+    (property "Value" "33k" (id 1) (at 141.097 62.0272 0)
       (effects (font (size 1.27 1.27)) (justify left))
     )
@@
       (effects (font (size 1.27 1.27)) (justify left))
     )
-    (property "Value" "33k" (id 1) (at 297.053 67.1072 0)
+    (property "Value" "10k" (id 1) (at 297.053 67.1072 0)
       (effects (font (size 1.27 1.27)) (justify left))
     )
@@
       (effects (font (size 1.27 1.27)) (justify left))
     )
-    (property "Value" "33k" (id 1) (at 86.868 48.0572 0)
+    (property "Value" "820k" (id 1) (at 86.868 48.0572 0)
       (effects (font (size 1.27 1.27)) (justify left))
     )
@@
       (effects (font (size 1.27 1.27)) (justify left))
     )
-    (property "Value" "18.7k±1%" (id 1) (at 294.132 205.5372 0)
+    (property "Value" "20k" (id 1) (at 294.132 205.5372 0)
       (effects (font (size 1.27 1.27)) (justify left))
     )
@@
       (effects (font (size 1.27 1.27)) (justify left))
     )
-    (property "Value" "18.7k±1%" (id 1) (at 177.927 59.4872 0)
+    (property "Value" "33k" (id 1) (at 177.927 59.4872 0)
       (effects (font (size 1.27 1.27)) (justify left))
     )
@@
       (effects (font (size 1.27 1.27)) (justify left))
     )
-    (property "Value" "18.7k±1%" (id 1) (at 169.037 77.9022 0)
+    (property "Value" "10k" (id 1) (at 169.037 77.9022 0)
       (effects (font (size 1.27 1.27)) (justify left))
     )
@@
     )
     (path "/4ccaa63b-7b0c-438b-bcee-d504e855bb86"
-      (reference "R2") (unit 1) (value "18.7k±1%") (footprint "Resistor_SMD:R_0402_1005Metric")
+      (reference "R2") (unit 1) (value "22k±1%") (footprint "Resistor_SMD:R_0402_1005Metric")
     )
     (path "/4f559366-c5b0-4ccd-8a02-2383450b8db6"
-      (reference "R3") (unit 1) (value "18.7k±1%") (footprint "Resistor_SMD:R_0402_1005Metric")
+      (reference "R3") (unit 1) (value "33k") (footprint "Resistor_SMD:R_0402_1005Metric")
     )
     (path "/13e44525-b5ff-48ec-bcda-86fa88213813"
-      (reference "R4") (unit 1) (value "18.7k±1%") (footprint "Resistor_SMD:R_0402_1005Metric")
+      (reference "R4") (unit 1) (value "10k") (footprint "Resistor_SMD:R_0402_1005Metric")
     )
     (path "/2bf9c215-a529-4aaa-84da-a7cd4c47ca6c"
@@
     )
     (path "/a695a885-0e66-40e4-9e87-c82b4f494866"
-      (reference "R14") (unit 1) (value "33k") (footprint "Resistor_SMD:R_0402_1005Metric")
+      (reference "R14") (unit 1) (value "820k") (footprint "Resistor_SMD:R_0402_1005Metric")
     )
     (path "/98689fbe-6a46-4c80-b994-7b262b0e1af4"
-      (reference "R15") (unit 1) (value "18.7k±1%") (footprint "Resistor_SMD:R_0402_1005Metric")
+      (reference "R15") (unit 1) (value "33k") (footprint "Resistor_SMD:R_0402_1005Metric")
     )
     (path "/ab17bd99-a805-41f9-9758-dffa330ed70e"
@@
     )
     (path "/9f9d1542-efd9-4176-85ed-571e1a3a85cb"
-      (reference "R17") (unit 1) (value "18.7k±1%") (footprint "Resistor_SMD:R_0402_1005Metric")
+      (reference "R17") (unit 1) (value "33k") (footprint "Resistor_SMD:R_0402_1005Metric")
     )
     (path "/587c7b95-ead5-46c5-ac8a-dffee84d24fa"
-      (reference "R18") (unit 1) (value "33k") (footprint "Resistor_SMD:R_0402_1005Metric")
+      (reference "R18") (unit 1) (value "820k") (footprint "Resistor_SMD:R_0402_1005Metric")
     )
     (path "/10a9aa63-6325-4aa9-98ba-e225c2be61e0"
@@
     )
     (path "/f7110e2c-ce36-4eb9-80f3-8af02c48b3b8"
-      (reference "R21") (unit 1) (value "18.7k±1%") (footprint "Resistor_SMD:R_0402_1005Metric")
+      (reference "R21") (unit 1) (value "10k") (footprint "Resistor_SMD:R_0402_1005Metric")
     )
     (path "/e3338377-42b4-42b2-956c-d5666e95543e"
-      (reference "R22") (unit 1) (value "18.7k±1%") (footprint "Resistor_SMD:R_0402_1005Metric")
+      (reference "R22") (unit 1) (value "33k") (footprint "Resistor_SMD:R_0402_1005Metric")
     )
     (path "/58528f2b-bdeb-4625-af95-471f2d6744b0"
@@
     )
     (path "/9eeb7860-1f43-4cce-a5e9-3432ab0652d7"
-      (reference "R30") (unit 1) (value "18.7k±1%") (footprint "Resistor_SMD:R_0402_1005Metric")
+      (reference "R30") (unit 1) (value "22k±1%") (footprint "Resistor_SMD:R_0402_1005Metric")
     )
     (path "/4a6ca347-374c-46e9-bf69-63f0ae4b3eb6"
@@
     )
     (path "/a4f1939a-cd19-4451-b6a7-b787d32e99e6"
-      (reference "R37") (unit 1) (value "33k") (footprint "Resistor_SMD:R_0402_1005Metric")
+      (reference "R37") (unit 1) (value "10k") (footprint "Resistor_SMD:R_0402_1005Metric")
     )
     (path "/49527bd6-d0da-445f-8bb9-b91afee1c513"
-      (reference "R38") (unit 1) (value "33k") (footprint "Resistor_SMD:R_0402_1005Metric")
+      (reference "R38") (unit 1) (value "10k") (footprint "Resistor_SMD:R_0402_1005Metric")
     )
     (path "/587dd1bc-5880-4e76-8990-407080bd294d"
@@
     )
     (path "/d9ea0679-1a4c-467a-8750-060458834648"
-      (reference "R41") (unit 1) (value "18.7k±1%") (footprint "Resistor_SMD:R_0402_1005Metric")
+      (reference "R41") (unit 1) (value "20k") (footprint "Resistor_SMD:R_0402_1005Metric")
     )
     (path "/0b6bd1aa-2e87-469c-ae0b-a0ea620bbf2c"
@@
     )
     (path "/928a705d-97eb-405f-b094-ff72d583ec4d"
-      (reference "R43") (unit 1) (value "33k") (footprint "Resistor_SMD:R_0402_1005Metric")
+      (reference "R43") (unit 1) (value "10k") (footprint "Resistor_SMD:R_0402_1005Metric")
     )
     (path "/b1330627-8c0a-44cd-91d7-af867c25c6d3"
