File: evaluation-boards/rf-switch-dpdt/rf-switch-dpdt.kicad_pcb (KiCad board)
At the start: 4 copper layers, 100 x 25 mm, 29 parts, among them J1 Conn_Coaxial, J10 Conn_Coaxial, J11 Conn_Coaxial, J12 Conn_Coaxial, J13 Conn_01x02, J14 Conn_01x02, J15 Conn_02x08_Odd_Even, J2 Conn_Coaxial, J3 Conn_Coaxial, J4 Conn_Coaxial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

Commit message: update CONSMA003.062 footprint
Other:
- board text added: "${TITLE} ${REVISION} ${ISSUE_DATE}"
- board text removed: "${TITLE} ${VERSION} ${DATE}"
