File: evaluation-boards/rf-switch-sp3t/rf-switch-sp3t.kicad_sch (KiCad schematic)
At the start: 33 parts, among them J1 Conn_Coaxial, J10 Conn_Coaxial, J11 Conn_Coaxial, J12 Conn_Coaxial, J13 Conn_01x02, J14 Conn_01x02, J15 Conn_02x06_Odd_Even, J2 Conn_Coaxial, J3 Conn_Coaxial, J4 Conn_Coaxial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

Commit message: Update RF test boards
- limiters
- rf-switch-spdt
- rf-switch-sp3t
Parts:
- C1, C10, C11, C12, C13, C14, C15, C2, C3, C4, C5, C6, C7, C8, C9: footprint Capacitor_SMD:C_0402_1005Metric -> Capacitor_SMD:C_0201_0603Metric
- J1, J10, J11, J12, J2, J3, J4, J5, J6, J7, J8, J9: footprint eval:CONSMA003.062 -> sma-variants:Linx_SMA_CONSMA003.062
