File: evaluation-boards/rf-switch-spdt/rf-switch-spdt.kicad_pcb (KiCad board)
At the start: 4 copper layers, 75 x 25 mm, 28 parts, among them J1 Conn_Coaxial, J13 Conn_01x02, J14 Conn_01x02, J15 Conn_02x04_Odd_Even, J2 Conn_Coaxial, J3 Conn_Coaxial, J4 Conn_Coaxial, J5 Conn_Coaxial, J6 Conn_Coaxial, J7 Conn_Coaxial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

Commit message: Update RF test boards
- limiters
- rf-switch-spdt
- rf-switch-sp3t
Parts:
- C1, C10, C11, C12, C13, C2, C3, C4, C5, C6, C7, C8, C9: footprint Capacitor_SMD:C_0402_1005Metric -> Capacitor_SMD:C_0201_0603Metric
- J1, J2, J3, J4, J5, J6, J7, J8, J9: footprint eval:CONSMA003.062 -> sma-variants:Linx_SMA_CONSMA003.062
- moved C2 0.42 mm to (118.6, 107.2)
- moved C1 0.42 mm to (115.8, 107.2)
- moved C12 0.32 mm to (161.1, 107.6)
- moved C9 0.32 mm to (164.0, 107.6)
- moved C4 0.30 mm to (134.7, 107.7)
- moved C7 0.30 mm to (131.3, 107.7)
- moved J2 0.10 mm to (110.0, 120.0)
- moved C13 0.08 mm to (107.0, 107.6)
Routing:
- net /V2: track 50.2 -> 44.0 mm
- net GND: track 11.0 -> 9.40 mm, vias 14 -> 41
- net Net-(U2-RFC): track 6.40 -> 5.35 mm
- net Net-(U3-INPUT): track 6.58 -> 5.78 mm
- net /V1: track 62.6 -> 61.8 mm
- net VCC: track 2.40 -> 1.68 mm
- added copper zone on B.Cu, net GND
- added copper zone on F.Cu, net GND
- removed copper zone on B.Cu, net (none)
- removed copper zone on F.Cu, net (none)
