File: evaluation-boards/trace-width/sma-jlcpcb.kicad_sch (KiCad schematic)
At the start: 34 parts, among them J1 Conn_Coaxial, J10 Conn_Coaxial, J11 Conn_Coaxial, J12 Conn_Coaxial, J13 Conn_Coaxial, J14 Conn_Coaxial, J15 Conn_Coaxial, J16 Conn_Coaxial, J17 Conn_Coaxial, J18 Conn_Coaxial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

Commit message: Update SMA connector board
Parts:
- removed J21, J22, J23, J24, J25, J26, J27, J28, J29, J30, J31, J32, J33, J34: Conn_Coaxial, symbol Connector:Conn_Coaxial
Other:
- moved on the sheet: J11, J12, J13, J14, J15, J16, J17, J18, J19, J20
