File: evaluation-boards/passives/passives.kicad_pcb (KiCad board)
At the start: 4 copper layers, 120 x 20 mm, 52 parts, among them J1 Conn_Coaxial, J10 Conn_Coaxial, J11 Conn_Coaxial, J12 Conn_Coaxial, J13 Conn_Coaxial, J14 Conn_Coaxial, J15 Conn_Coaxial, J16 Conn_Coaxial, J17 Conn_Coaxial, J18 Conn_Coaxial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

Commit message: Update passives board
Parts:
- added C19: C, Capacitor_SMD:C_0201_0603Metric, F.Cu at (193.3, 111.2)
- added C20: C, Capacitor_SMD:C_0201_0603Metric, F.Cu at (203.8, 111.2)
- added J25: Conn_01x02_Pin, Connector_PinHeader_2.54mm:PinHeader_1x02_P2.54mm_Vertical, F.Cu at (175.0, 111.3)
- added J26: Conn_01x02_Pin, Connector_PinHeader_2.54mm:PinHeader_1x02_P2.54mm_Vertical, F.Cu at (193.7, 106.3)
- C1, C10, C12, C13, C14, C15, C2, C4, C5, C9: footprint Capacitor_SMD:C_0402_1005Metric_Pad0.74x0.62mm_HandSolder -> Capacitor_SMD:C_0201_0603Metric
- C11: footprint Capacitor_SMD:C_0603_1608Metric_Pad1.08x0.95mm_HandSolder -> Capacitor_SMD:C_0201_0603Metric
- C16: footprint Capacitor_SMD:C_0805_2012Metric_Pad1.18x1.45mm_HandSolder -> Capacitor_SMD:C_0402_1005Metric
- C17, C18, C6, C7, C8: footprint Capacitor_SMD:C_0402_1005Metric_Pad0.74x0.62mm_HandSolder -> Capacitor_SMD:C_0402_1005Metric
- C3: footprint Capacitor_SMD:C_0201_0603Metric_Pad0.64x0.40mm_HandSolder -> Capacitor_SMD:C_0201_0603Metric
- J1, J10, J11, J12, J13, J14, J15, J16, J17, J18, J19, J2, J20, J21, J22, J23, J24, J3, J4, J5, J6, J7, J8, J9: footprint passives:SMA-EDGE -> sma-variants:Linx_SMA_CONSMA003.062
- L1, L3, L5: footprint Capacitor_SMD:C_0201_0603Metric_Pad0.64x0.40mm_HandSolder -> Inductor_SMD:L_0201_0603Metric
- L10: footprint Capacitor_SMD:C_0805_2012Metric_Pad1.18x1.45mm_HandSolder -> Inductor_SMD:L_0402_1005Metric
- L2: footprint Capacitor_SMD:C_0201_0603Metric_Pad0.64x0.40mm_HandSolder -> Inductor_SMD:L_0603_1608Metric
- L4, L8: footprint Capacitor_SMD:C_0402_1005Metric_Pad0.74x0.62mm_HandSolder -> Inductor_SMD:L_0402_1005Metric
- L6, L9: footprint Capacitor_SMD:C_0402_1005Metric_Pad0.74x0.62mm_HandSolder -> Inductor_SMD:L_0603_1608Metric
- L7: footprint Capacitor_SMD:C_0603_1608Metric_Pad1.08x0.95mm_HandSolder -> Inductor_SMD:L_0201_0603Metric
- moved C1 1.90 mm to (180.0, 108.9)
- moved C10 1.90 mm to (190.0, 111.1)
- moved C12 1.90 mm to (160.0, 108.9)
- moved C13 1.90 mm to (160.0, 111.1)
- moved C2 1.90 mm to (180.0, 111.1)
- moved C4 1.90 mm to (130.0, 108.9)
- moved C5 1.90 mm to (130.0, 111.1)
- moved C9 1.90 mm to (190.0, 108.9)
- moved C14 1.80 mm to (200.0, 108.8)
- moved C15 1.80 mm to (200.0, 111.2)
- moved C17 1.60 mm to (170.0, 108.6)
- moved C18 1.60 mm to (170.0, 111.4)
- moved C7 1.60 mm to (140.0, 108.6)
- moved C8 1.60 mm to (140.0, 111.4)
- moved L7 0.70 mm to (160.3, 110.0)
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Connections:
- L6 pad 2: GND -> VCC
- L9 pad 2: GND -> VCC
Routing:
- net GND: track 8.37 -> 3.72 mm, vias 7 -> 34
- net VCC: track 0.00 -> 3.72 mm, vias 0 -> 2
- net Net-(C12-Pad2): track 4.98 -> 1.58 mm
- net Net-(C10-Pad1): track 4.94 -> 1.58 mm
- net Net-(C1-Pad2): track 4.94 -> 1.58 mm
- net Net-(C4-Pad2): track 4.94 -> 1.58 mm
- net Net-(C14-Pad2): track 4.92 -> 1.77 mm
- net Net-(C7-Pad2): track 4.96 -> 1.85 mm
- net Net-(C17-Pad2): track 4.90 -> 1.85 mm
- net Net-(J8-In): track 4.30 -> 6.45 mm
- net Net-(J7-In): track 4.30 -> 6.45 mm
- net Net-(J4-In): track 4.30 -> 6.45 mm
- net Net-(J3-In): track 4.30 -> 6.45 mm
- net Net-(J18-In): track 4.30 -> 6.45 mm
- net Net-(J17-In): track 4.30 -> 6.45 mm
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- added copper zone on B.Cu, net GND
- added copper zone on F.Cu, net GND
- added copper zone on In2.Cu, net VCC
Other:
- board text added: "GND"
- board text added: "VCC"
- board text added: "a-p"
- board text added: "anti-pads"
- board text added: "passives 2024-11-03"
- board text removed: "passives 2022-04-08"

Commit message: Update passives board
Parts:
- removed C17, C18: C, Capacitor_SMD:C_0402_1005Metric
- removed C19, C20: C, Capacitor_SMD:C_0201_0603Metric
- removed J13, J14, J19, J20: Conn_Coaxial, sma-variants:Linx_SMA_CONSMA003.062
- removed L10: L, Inductor_SMD:L_0402_1005Metric
- removed L9: L, Inductor_SMD:L_0603_1608Metric
- added L11: L, Inductor_SMD:L_0603_1608Metric, F.Cu at (150.8, 110.0)
- added L12: L, Inductor_SMD:L_0603_1608Metric, F.Cu at (163.8, 110.0)
- added R1: R, Resistor_SMD:R_0402_1005Metric, F.Cu at (160.5, 108.8)
- added R10: R, Resistor_SMD:R_0201_0603Metric, F.Cu at (93.1, 110.0)
- added R11: R, Resistor_SMD:R_0201_0603Metric, F.Cu at (92.8, 107.5)
- added R2: R, Resistor_SMD:R_0402_1005Metric, F.Cu at (163.5, 108.8)
- added R3: R, Resistor_SMD:R_0402_1005Metric, F.Cu at (163.0, 107.4)
- added R4: R, Resistor_SMD:R_0201_0603Metric, F.Cu at (180.3, 109.7)
- added R5: R, Resistor_SMD:R_0201_0603Metric, F.Cu at (182.0, 111.0)
- added R6: R, Resistor_SMD:R_0201_0603Metric, F.Cu at (181.3, 112.5)
- added R7: R, Resistor_SMD:R_0201_0603Metric, F.Cu at (183.1, 111.4)
- added R8: R, Resistor_SMD:R_0201_0603Metric, F.Cu at (94.2, 109.7)
- added R9: R, Resistor_SMD:R_0201_0603Metric, F.Cu at (91.7, 109.3)
- C12: footprint Capacitor_SMD:C_0201_0603Metric -> Capacitor_SMD:C_0402_1005Metric
- C8: footprint Capacitor_SMD:C_0402_1005Metric -> Capacitor_SMD:C_0201_0603Metric
- L2, L6: footprint Inductor_SMD:L_0603_1608Metric -> Inductor_SMD:L_0805_2012Metric
- L3, L7: footprint Inductor_SMD:L_0201_0603Metric -> Inductor_SMD:L_0603_1608Metric
- L4: footprint Inductor_SMD:L_0402_1005Metric -> Inductor_SMD:L_0805_2012Metric
- L8: footprint Inductor_SMD:L_0402_1005Metric -> Inductor_SMD:L_0201_0603Metric
- moved L8 110.2 mm to (90.3, 110.0)
- moved C15 110.0 mm to (90.0, 113.3)
- moved C14 107.3 mm to (92.8, 109.0)
- moved L6 99.4 mm to (93.1, 111.2)
- moved L5 98.6 mm to (91.7, 110.0)
- moved J26 88.9 mm to (105.0, 111.3), turned to 180 degrees
- moved C13 65.2 mm to (94.8, 109.7), turned to 90 degrees
- moved J25 60.0 mm to (115.0, 111.3)
- moved C8 42.4 mm to (182.3, 112.1), turned to 90 degrees
- moved C4 30.1 mm to (160.0, 106.4)
- moved C5 30.1 mm to (160.0, 113.3)
- moved C7 24.8 mm to (164.6, 111.7), turned to 90 degrees
- moved C10 10.3 mm to (180.0, 113.4)
- moved C1 9.76 mm to (170.3, 110.0), turned to 180 degrees
- moved C9 9.39 mm to (180.9, 111.4), turned to 90 degrees
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Connections:
- C1 pad 1: Net-(J3-In) -> GND
- C1 pad 2: Net-(C1-Pad2) -> Net-(J23-In)
- C10 pad 2: Net-(J14-In) -> Net-(J4-In)
- C11 pad 1: Net-(J15-In) -> GND
- C11 pad 2: Net-(J16-In) -> Net-(J15-In)
- C12 pad 1: Net-(J17-In) -> GND
- C13 pad 1: Net-(C12-Pad2) -> GND
- C13 pad 2: Net-(J18-In) -> Net-(C13-Pad2)
- C15 pad 1: Net-(C14-Pad2) -> Net-(C15-Pad1)
- C15 pad 2: Net-(J20-In) -> Net-(J6-In)
- C16 pad 1: Net-(J21-In) -> GND
- C16 pad 2: Net-(J22-In) -> Net-(J21-In)
- C2 pad 1: Net-(C1-Pad2) -> Net-(J3-In)
- C2 pad 2: Net-(J4-In) -> Net-(C10-Pad1)
- C3 pad 2: Net-(J6-In) -> Net-(C15-Pad1)
- C4 pad 1: Net-(J7-In) -> Net-(J17-In)
- C5 pad 2: Net-(J8-In) -> Net-(J18-In)
- C7 pad 1: Net-(J11-In) -> GND
- C7 pad 2: Net-(C7-Pad2) -> VCC
- C8 pad 1: Net-(C7-Pad2) -> GND
- C8 pad 2: Net-(J12-In) -> Net-(C8-Pad2)
- C9 pad 2: Net-(C10-Pad1) -> Net-(C9-Pad2)
- J12 pad 1: Net-(J12-In) -> Net-(J11-In)
- J16 pad 1: Net-(J16-In) -> Net-(J15-In)
- J22 pad 1: Net-(J22-In) -> Net-(J21-In)
- J24 pad 1: Net-(J24-In) -> Net-(J23-In)
- J8 pad 1: Net-(J8-In) -> Net-(J7-In)
- L1 pad 1: Net-(C1-Pad2) -> Net-(C10-Pad1)
- L1 pad 2: Net-(L1-Pad2) -> Net-(C9-Pad2)
- L2 pad 1: Net-(L1-Pad2) -> Net-(C9-Pad2)
- L2 pad 2: GND -> VCC
- L3 pad 1: Net-(C4-Pad2) -> Net-(J7-In)
- L4 pad 1: Net-(C7-Pad2) -> Net-(J11-In)
- L5 pad 1: Net-(C10-Pad1) -> Net-(L5-Pad1)
- L5 pad 2: Net-(L5-Pad2) -> Net-(C14-Pad2)
- L6 pad 1: Net-(L5-Pad2) -> Net-(C14-Pad2)
- L7 pad 1: Net-(C12-Pad2) -> Net-(C4-Pad2)
- L7 pad 2: GND -> Net-(L12-Pad1)
- L8 pad 1: Net-(C14-Pad2) -> Net-(C15-Pad1)
- L8 pad 2: Net-(L8-Pad2) -> Net-(L5-Pad1)
Routing:
- net GND: track 3.72 -> 15.8 mm, vias 34 -> 35
- net Net-(J23-In): track 5.99 -> 15.7 mm
- net Net-(J11-In): track 5.99 -> 15.7 mm
- net Net-(J7-In): track 6.45 -> 15.7 mm
- net Net-(J21-In): track 7.39 -> 15.7 mm
- net Net-(J15-In): track 7.55 -> 15.7 mm
- net Net-(J16-In): track 7.55 -> 0.00 mm
- net Net-(J22-In): track 7.39 -> 0.00 mm
- net Net-(C15-Pad1): track 0.00 -> 6.68 mm
- net Net-(J8-In): track 6.45 -> 0.00 mm
- net Net-(J14-In): track 6.45 -> 0.00 mm
- net Net-(J20-In): track 6.35 -> 0.00 mm
- net Net-(J24-In): track 5.99 -> 0.00 mm
- net Net-(J12-In): track 5.99 -> 0.00 mm
- net Net-(C9-Pad1): track 6.45 -> 0.74 mm
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Other:
- board size 120 x 20 mm -> 100 x 20 mm
- board text added: "passives 2024-12-08"
- board text removed: "a-p"
- board text removed: "anti-pads"
- board text removed: "passives 2024-11-03"
