File: evaluation-boards/passives/passives.kicad_sch (KiCad schematic)
At the start: 52 parts

Commit message: Update passives board
Parts:
- added C19, C20: C, Capacitor_SMD:C_0201_0603Metric, symbol Device:C
- added J25, J26: Conn_01x02_Pin, Connector_PinHeader_2.54mm:PinHeader_1x02_P2.54mm_Vertical, symbol Connector:Conn_01x02_Pin
- C1, C10, C11, C12, C13, C14, C15, C2, C3, C4, C5, C9: value (none) -> C; footprint (none) -> Capacitor_SMD:C_0201_0603Metric
- C16, C17, C18, C6, C7, C8: value (none) -> C; footprint (none) -> Capacitor_SMD:C_0402_1005Metric
- J1, J10, J11, J12, J13, J14, J15, J16, J17, J18, J19, J2, J20, J21, J22, J23, J24, J3, J4, J5, J6, J7, J8, J9: value (none) -> Conn_Coaxial; footprint (none) -> sma-variants:Linx_SMA_CONSMA003.062
- L1, L3, L5, L7: value (none) -> L; footprint (none) -> Inductor_SMD:L_0201_0603Metric
- L10, L4, L8: value (none) -> L; footprint (none) -> Inductor_SMD:L_0402_1005Metric
- L2, L6, L9: value (none) -> L; footprint (none) -> Inductor_SMD:L_0603_1608Metric
Connections:
- net GND: now also C19.1, C20.1, J26.1 (Pin_1), J26.2 (Pin_2); no longer L6.2, L9.2
- new net VCC: C19.2, C20.2, J25.1 (Pin_1), J25.2 (Pin_2), L6.2, L9.2
Other:
- moved on the sheet: C14, C15, J19, J20, L8, L9

Commit message: Update passives board
Parts:
- removed C17, C18: C, Capacitor_SMD:C_0402_1005Metric, symbol Device:C
- removed C19, C20: C, Capacitor_SMD:C_0201_0603Metric, symbol Device:C
- removed J13, J14, J19, J20: Conn_Coaxial, sma-variants:Linx_SMA_CONSMA003.062, symbol Connector:Conn_Coaxial
- removed L10: L, Inductor_SMD:L_0402_1005Metric, symbol Device:L
- removed L9: L, Inductor_SMD:L_0603_1608Metric, symbol Device:L
- added L11, L12: L, Inductor_SMD:L_0603_1608Metric, symbol Device:L
- added R1, R2, R3: R, Resistor_SMD:R_0402_1005Metric, symbol Device:R
- added R10, R11, R4, R5, R6, R7, R8, R9: R, Resistor_SMD:R_0201_0603Metric, symbol Device:R
- C12: footprint Capacitor_SMD:C_0201_0603Metric -> Capacitor_SMD:C_0402_1005Metric
- C8: footprint Capacitor_SMD:C_0402_1005Metric -> Capacitor_SMD:C_0201_0603Metric
- L2, L6: footprint Inductor_SMD:L_0603_1608Metric -> Inductor_SMD:L_0805_2012Metric
- L3, L7: footprint Inductor_SMD:L_0201_0603Metric -> Inductor_SMD:L_0603_1608Metric
- L4: footprint Inductor_SMD:L_0402_1005Metric -> Inductor_SMD:L_0805_2012Metric
- L8: footprint Inductor_SMD:L_0402_1005Metric -> Inductor_SMD:L_0201_0603Metric
Connections:
- net GND: now also C1.1, C11.1, C12.1, C13.1, C16.1, C7.1, C8.1, L11.2, R11.2, R6.2; no longer L2.2, L7.2
- net VCC: now also C7.2, L2.2, L12.2, R10.2, R2.2, R5.2, R7.1, R8.1
- net at C14.1: now also R11.1
- net at C15.1, L8.1: now also C3.2; no longer C14.2
- net at J23.1 (In): now also C1.2, J24.1 (In)
- net at J6.1 (In): now also C15.2; no longer C3.2
- net at C4.2, C5.1: now also L7.1, R1.1; no longer L3.1
- net at J7.1 (In): now also J8.1 (In), L3.1; no longer C4.1
- net at C5.2: now also J18.1 (In); no longer J8.1 (In)
- net at J21.1 (In): now also C16.2, J22.1 (In); no longer C16.1
- net at J15.1 (In): now also C11.2, J16.1 (In); no longer C11.1
- net at L1.2, L2.1: now also C9.2, R4.2, R5.1
- net at L8.2: now also L5.1, R9.1
- net at J11.1 (In): now also J12.1 (In), L4.1; no longer C7.1
- net at C10.2: now also J4.1 (In)
- net at C13.2: now also R8.2; no longer J18.1 (In)
- net at J3.1 (In): now also C2.1; no longer C1.1
- net at J1.1 (In), J2.1 (In): now also L11.1
- net at J17.1 (In): now also C4.1; no longer C12.1
- net at C9.1: now also R6.1
- net at L5.2, L6.1: now also C14.2, R10.1, R9.2
- net at C2.2: now also C10.1, L1.1, R4.1; no longer J4.1 (In)
- net at C8.2: now also R7.2; no longer J12.1 (In)
- new net: L12.1, L7.2, R1.2, R2.1, R3.1
- new net: C12.2, R3.2
Other:
- moved on the sheet: C11, C16, C3, J11, J12, J17, J18, J2, J23, J24, J4, J5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
