File: evaluation-boards/limiters/limiters.kicad_sch (KiCad schematic)
At the start: 132 parts

Commit message: Update RF test boards
- limiters
- rf-switch-spdt
- rf-switch-sp3t
Parts:
- removed C14, C15, C16, C19, C20, C25, C26, C27, C28, C29, C30, C33, C34, C35, C36, C39: (no value), symbol Device:C
- removed D10, D20, D21, D23, D26, D27: (no value), symbol Device:D
- removed D11, D12, D15, D16, D17, D18, D19, D6: (no value), symbol Device:D_Schottky
- removed D24, D25: (no value), symbol limiters:D_AKA
- removed D3, D4: (no value), symbol Device:D_Schottky_Dual_Series_AKC
- removed J11, J12, J13, J14, J17, J18, J23, J24, J25, J26, J27, J28, J3, J31, J32, J33, J34, J4, J5, J6: (no value), symbol Connector:Conn_Coaxial
- removed L11, L12, L14, L15, L16, L17, L19, L6, L7, L8, L9: (no value), symbol Device:L
- removed R3, R4: (no value), symbol Device:R
- removed TP1, TP2: (no value), symbol Connector:TestPoint
- removed U1: (no value), symbol gsg-symbols:SKY13453
- added C40, C41, C42, C43, C44, C46, C47, C52, C63, C64, C68, C69, C71, C72, C73, C74, C75: 1 uF, Capacitor_SMD:C_0201_0603Metric, symbol Device:C
- added C65, C66, C67, C70: 220 nF, Capacitor_SMD:C_0201_0603Metric, symbol Device:C
- added D29, D31, D37, D4, D41: PIN, Diode_SMD:D_0201_0603Metric, symbol Device:D
- added D3, D30, D32, D38, D42: Schottky, Diode_SMD:D_0201_0603Metric, symbol Device:D_Schottky
- added D33, D34, D35: LED, LED_SMD:LED_0603_1608Metric, symbol Device:LED
- added D39: PIN, limiters:SMP1345-087LF, symbol Device:D
- added J39, J40, J41, J42, J47, J48, J49, J50, J51, J52, J53, J54: Conn_Coaxial, sma-variants:Linx_SMA_CONSMA003.062, symbol Connector:Conn_Coaxial
- added L21, L24, L25, L28, L35, L39, L40, L43: 0.5 nH, Inductor_SMD:L_0201_0603Metric, symbol Device:L
- added L22, L26, L29, L37, L41, L44: 47uH, Inductor_SMD:L_0603_1608Metric, symbol Device:L
- added L23, L27, L30, L38, L42, L45: 33nH, Inductor_SMD:L_0201_0603Metric, symbol Device:L
- added L46: 1 nH, Inductor_SMD:L_0201_0603Metric, symbol Device:L
- added Q1, Q2, Q3: NPN+PNP, Package_TO_SOT_SMD:SOT-363_SC-70-6, symbol Device:Q_Dual_NPN_PNP_E1B1C2E2B2C1
- added R10, R12, R14, R16, R17, R19, R20, R40, R42, R44, R49, R52, R53, R7, R8: 1k, Resistor_SMD:R_0402_1005Metric, symbol Device:R
- added R11, R38, R39, R48: 0, Resistor_SMD:R_0402_1005Metric, symbol Device:R
- added R13, R15, R18, R36, R37, R41, R43, R45, R46, R47, R5, R51, R54, R6, R9: 10k, Resistor_SMD:R_0402_1005Metric, symbol Device:R
- added R50: 3.3k, Resistor_SMD:R_0402_1005Metric, symbol Device:R
- C1, C13, C2, C3, C7, C8: value (none) -> 1 uF; footprint (none) -> Capacitor_SMD:C_0201_0603Metric; Part Number GRM033R61A224KE90D -> GRM033R61A105ME44D
- C10, C11, C12, C17, C18, C21, C22, C23, C24, C31, C32, C37, C38, C9: value (none) -> 220 nF; footprint (none) -> Capacitor_SMD:C_0201_0603Metric
- C4: value (none) -> 1 uF; footprint (none) -> Capacitor_SMD:C_0201_0603Metric; Note DNP -> (none); Part Number GRM033R61A224KE90D -> GRM033R61A105ME44D
- C5: value (none) -> 1 uF; footprint (none) -> Capacitor_SMD:C_0201_0603Metric; Manufacturer (none) -> Murata; Part Number (none) -> GRM033R61A105ME44D
- C6: value (none) -> 1 uF; footprint (none) -> Capacitor_SMD:C_0201_0603Metric; Manufacturer (none) -> Murata; Note DNP -> (none); Part Number (none) -> GRM033R61A105ME44D
- D1, D14, D22: value (none) -> PIN; footprint (none) -> limiters:SMP1345-087LF
- D13, D9: value (none) -> PIN; footprint (none) -> limiters:SMP1304-085LF
- D2: value (none) -> Schottky; footprint (none) -> Diode_SMD:D_0201_0603Metric; Manufacturer Toshibar -> Infineon; Part Number JDH2S02FSTPL3 -> BAT2402LSE6327XTSA1; Substitution Skyworks SMS7621-040LF, Infineon BAT1502LRHE6327XTSA1r -> Rochester BAT6202LSE6327, Toshiba JDH2S02SL,L3F, onsemi NSR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
- D28: value (none) -> Dual_PIN; footprint (none) -> Package_TO_SOT_SMD:SOT-23
- D5: value (none) -> PIN; footprint (none) -> Diode_SMD:D_0201_0603Metric; Manufacturer onsemi -> Infineon; Part Number NSDP301MX3T5G -> BAR9002ELSE6327XTSA1; Substitution (none) -> Toshiba JDP2S08SC
- D7: value (none) -> PIN; footprint (none) -> Diode_SMD:D_0201_0603Metric
- D8: value (none) -> Schottky; footprint (none) -> Diode_SMD:D_0201_0603Metric
- J1, J2: value (none) -> Conn_01x02; footprint (none) -> Connector_PinHeader_2.54mm:PinHeader_1x02_P2.54mm_Vertical
- J10, J15, J16, J19, J20, J21, J22, J29, J30, J35, J36, J37, J38, J7, J8, J9: value (none) -> Conn_Coaxial; footprint (none) -> sma-variants:Linx_SMA_CONSMA003.062
- L1, L4: value (none) -> 33nH; footprint (none) -> Inductor_SMD:L_0201_0603Metric; Manufacturer Taiyo Yuden -> Murata; Part Number BRL1608T100M -> LQP03TN33NJ02D
- L10: value (none) -> 0.6 nH; footprint (none) -> Inductor_SMD:L_0201_0603Metric
- L13: value (none) -> 0.5 nH; footprint (none) -> Inductor_SMD:L_0201_0603Metric; Part Number LQP03HQ0N4W02D -> LQP03HQ0N5W02D
- L18: value (none) -> 0.8 nH; footprint (none) -> Inductor_SMD:L_0201_0603Metric
- L2: value (none) -> 47uH; footprint (none) -> Inductor_SMD:L_0603_1608Metric; Manufacturer Murata -> Taiyo Yuden; Part Number LQP03HQ0N4W02D -> LSQNB160808T470M; Substitution (none) -> LSQNB160808T470K
- L20: value (none) -> 1.4 nH; footprint (none) -> Inductor_SMD:L_0201_0603Metric
- L3: value (none) -> 1.0 nH; footprint (none) -> Inductor_SMD:L_0201_0603Metric
- L5: value (none) -> 47uH; footprint (none) -> Inductor_SMD:L_0603_1608Metric; Manufacturer Murata -> Taiyo Yuden; Part Number LQP03HQ1N4W02D -> LSQNB160808T470M; Substitution (none) -> LSQNB160808T470K
- R1: value (none) -> 1k; footprint (none) -> Resistor_SMD:R_0402_1005Metric
- R2: value (none) -> 10k; footprint (none) -> Resistor_SMD:R_0402_1005Metric; Note DNP -> (none); now not fitted
Connections:
- net GND: now also C1.2, C13.2, C2.2, C3.2, C4.2, C5.2, C7.2, C8.2, L2.2, L5.2, C42.2, C43.2, C46.2, C64.2, C68.2, C71.2, C73.2, C74.2, D3.2 (A), D31.1 (K), D33.1 (K), D34.1 (K), D35.1 (K), D39.1 (K), J39.2 (Ext), J40.2 (Ext), J41.2 (Ext), J42.2 (Ext), J47.2 (Ext), J48.2 (Ext), J49.2 (Ext), J50.2 (Ext), J51.2 (Ext), J52.2 (Ext), J53.2 (Ext), J54.2 (Ext), L22.2, L26.2, L44.2, Q1.2 (B1), Q2.1 (E1), Q3.1 (E1), R13.2, R18.2, R36.2, R40.2, R42.2, R44.2, R47.2, R49.2, R5.2, R54.2, R9.2; no longer C5.1, D5.1 (K), L4.2, R2.2
- net VCC: now also C13.1, C2.1, C3.1, C4.1, C5.1, C6.1, C7.1, C8.1, R2.2, Q1.4 (E2), Q2.4 (E2), Q3.4 (E2), R15.1, R37.1, R41.2, R43.2, R45.1, R46.1, R51.1, R6.1; no longer C5.2
- net at C11.1, C12.2, D1.2 (A): now also L1.1; no longer L4.1
- net at C1.1: now also R1.1, R2.1, D4.2 (A)
- net at C18.2, D9.3 (A): now also L4.1
- net at L5.1: now also L4.2
- net at C24.2, L13.1: now also D3.1 (K)
- net at C22.2, L10.1: now also D2.1 (K)
- net at C32.2, L18.1: now also D4.1 (K)
- net at L2.1: now also L1.2; no longer C8.2
- new net: C67.1, D5.1 (K), L40.2
- new net: C67.2, J51.1 (In)
- new net: L35.1, L38.1, L39.2
- new net: L37.1, L38.2
- new net: D33.2 (A), R12.1
- new net: C41.1, J40.1 (In)
- new net: L41.2, R40.1, R41.1
- new net: C40.1, D29.1 (K), L24.2
- new net: C42.1, D29.2 (A), R11.1
- new net: C44.2, J41.1 (In)
- new net: R39.2, R46.2, R47.1, R48.1
- new net: C41.2, D30.1 (K), L21.1
- new net: Q3.5 (B2), R51.2, R52.1
- new net: C40.2, J39.1 (In)
- new net: C71.1, D5.2 (A), R42.1, R43.1
- new net: C75.1, J54.1 (In)
- new net: C64.1, D37.2 (A), R39.1
- new net: C52.1, L27.1, L28.2
- new net: L26.1, L27.2
- new net: C73.1, D41.2 (A), R49.1, R50.1
- new net: Q3.3 (C2), R20.2, R50.2
- new net: C68.1, D38.1 (K), R38.2
- new net: C52.2, L25.1, L30.1
- new net: C63.1, D37.1 (K), L35.2
- new net: C65.1, D39.2 (A), L43.2
- new net: C65.2, J49.1 (In)
- new net: L21.2, L23.1, L24.1
- new net: C70.1, J52.1 (In)
- new net: C72.2, J53.1 (In)
- new net: Q1.1 (E1), R5.1, R7.2
- new net: Q1.6 (C1), R8.2
- new net: D34.2 (A), R19.1
- new net: C74.1, D42.1 (K), R53.1
- new net: C75.2, D42.2 (A), L46.1
- new net: R10.1, R11.2, R9.1
- new net: C63.2, J47.1 (In)
- new net: C47.1, J42.1 (In)
- new net: C47.2, D32.2 (A), L28.1
- new net: C66.2, L42.1, L43.1
- new net: C43.1, D30.2 (A), R7.1
- new net: C69.2, D38.2 (A), L39.1
- new net: R36.1, R37.2, R38.1, R48.2
- new net: C72.1, D41.1 (K), L46.2
- new net: Q2.2 (B1), R17.2, R18.1
- new net: Q2.6 (C1), R16.2
- new net: C46.1, D32.1 (K), R17.1
- new net: Q1.3 (C2), R10.2, R12.2
- new net: L29.2, R13.1, R14.1
- new net: L44.1, L45.2
- new net: L29.1, L30.2
- new net: C66.1, J50.1 (In)
- new net: Q1.5 (B2), R6.2, R8.1
- new net: C44.1, D31.2 (A), L25.2
- new net: Q2.3 (C2), R14.2, R19.2
- new net: L37.2, R44.1, R45.2
- new net: C70.2, L40.1, L45.1
- new net: D35.2 (A), R20.1
- new net: Q2.5 (B2), R15.2, R16.1
- new net: Q3.2 (B1), R53.2, R54.1
- new net: C69.1, J48.1 (In)
- new net: L41.1, L42.2
- new net: Q3.6 (C1), R52.2
- new net: L22.1, L23.2
Other:
- note added: "Active PIN-Schottky"
- note added: "Biased PIN"
- note added: "Biased PIN-Schottky"
- note removed: "Schottky-Schottky"
- note removed: "Schottky-switch"
- moved on the sheet: C10, C11, C12, C17, C18, C21, C22, C23, C24, C31, C32, C37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

Commit message: Update limiters board
Parts:
- removed C37, C38, C65, C66: 220 nF, Capacitor_SMD:C_0201_0603Metric, symbol Device:C
- removed C40, C41, C42, C43, C44, C46, C47, C52, C72, C73, C74, C75: 1 uF, Capacitor_SMD:C_0201_0603Metric, symbol Device:C
- removed D13, D9: PIN, limiters:SMP1304-085LF, symbol limiters:D_AKA
- removed D22, D39: PIN, limiters:SMP1345-087LF, symbol Device:D
- removed D28: Dual_PIN, Package_TO_SOT_SMD:SOT-23, symbol Device:D_Dual_Series_AKC
- removed D29, D31, D41: PIN, Diode_SMD:D_0201_0603Metric, symbol Device:D
- removed D3, D30, D32, D42: Schottky, Diode_SMD:D_0201_0603Metric, symbol Device:D_Schottky
- removed D33, D34, D35: LED, LED_SMD:LED_0603_1608Metric, symbol Device:LED
- removed J16, J19, J20, J21, J22, J29, J30, J35, J36, J39, J40, J41, J42, J49, J50, J53, J54, J9: Conn_Coaxial, sma-variants:Linx_SMA_CONSMA003.062, symbol Connector:Conn_Coaxial
- removed L10: 0.6 nH, Inductor_SMD:L_0201_0603Metric, symbol Device:L
- removed L13, L21, L24, L25, L28, L35, L39, L40, L43: 0.5 nH, Inductor_SMD:L_0201_0603Metric, symbol Device:L
- removed L18: 0.8 nH, Inductor_SMD:L_0201_0603Metric, symbol Device:L
- removed L20: 1.4 nH, Inductor_SMD:L_0201_0603Metric, symbol Device:L
- removed L22, L26, L29, L37, L41, L44: 47uH, Inductor_SMD:L_0603_1608Metric, symbol Device:L
- removed L23, L27, L30, L38, L42, L45: 33nH, Inductor_SMD:L_0201_0603Metric, symbol Device:L
- removed L46: 1 nH, Inductor_SMD:L_0201_0603Metric, symbol Device:L
- removed Q1, Q2, Q3: NPN+PNP, Package_TO_SOT_SMD:SOT-363_SC-70-6, symbol Device:Q_Dual_NPN_PNP_E1B1C2E2B2C1
- removed R18, R45, R51, R54: 10k, Resistor_SMD:R_0402_1005Metric, symbol Device:R
- removed R19, R20, R44, R49, R52, R53: 1k, Resistor_SMD:R_0402_1005Metric, symbol Device:R
- removed R50: 3.3k, Resistor_SMD:R_0402_1005Metric, symbol Device:R
- added C14, C25, C26: C, Capacitor_SMD:C_0201_0603Metric, symbol Device:C
- added C15, C19, C20, C27, C28, C29, C30, C33, C34, C35: 1 uF, Capacitor_SMD:C_0201_0603Metric, symbol Device:C
- added C16: 1 uF, Capacitor_SMD:C_0402_1005Metric, symbol Device:C
- added D10, D12, D3: PIN, eval:TSLP-2-19, symbol Device:D
- added D11, D13, D6, D9: Schottky, eval:TSSLP-2-1, symbol Device:D_Schottky
- added J11, J12, J13, J14, J17, J18, J3, J4, J5, J6: Conn_Coaxial, sma-variants:Linx_SMA_CONSMA003.062, symbol Connector:Conn_Coaxial
- added J16, J19, J9: Conn_01x02, Connector_PinHeader_2.54mm:PinHeader_1x02_P2.54mm_Vertical, symbol Connector_Generic:Conn_01x02
- added L6: 1.0 nH, Inductor_SMD:L_0201_0603Metric, symbol Device:L
- added L7: L, Inductor_SMD:L_0805_2012Metric, symbol Device:L
- added L8, L9: L, Inductor_SMD:L_0201_0603Metric, symbol Device:L
- added Q1, Q2, Q4: NMOS/PMOS, Package_TO_SOT_SMD:SOT-563, symbol eval:Q_Dual_NMOS_PMOS_S1G1D2S2G2D1
- added R21, R22, R3, R4: R, Resistor_SMD:R_0201_0603Metric, symbol Device:R
- added R23, R24, R25, R27, R28, R29, R30, R31, R32, R34, R55, R56, R57: 10k, Resistor_SMD:R_0402_1005Metric, symbol Device:R
- added R33, R58: 3.3k, Resistor_SMD:R_0402_1005Metric, symbol Device:R
- added R35: 0, Resistor_SMD:R_0402_1005Metric, symbol Device:R
- added U1: MADL-011021-14150T, eval:TDFN-6-1EP_1.5x1.2mm_P0.4mm_EP0.47x0.8mm, symbol eval:MADL-011021-14150T
- added U2: LMV358, Package_SO:MSOP-8_3x3mm_P0.65mm, symbol Amplifier_Operational:LMV358
- C10, C12, C17, C18, C21, C24, C32, C67, C70: value 220 nF -> 1 uF; Part Number GRM033R61A224KE90D -> GRM033R61A105ME44D
- C11, C22: value 220 nF -> C; Manufacturer Murata -> (none); Part Number GRM033R61A224KE90D -> (none)
- C2, C71, R13, R43, R9: now not fitted
- C23: value 220 nF -> C; Manufacturer Murata -> (none); Part Number GRM033R61A224KE90D -> (none); now not fitted
- C31: value 220 nF -> 1 uF; footprint Capacitor_SMD:C_0201_0603Metric -> Capacitor_SMD:C_0402_1005Metric; Manufacturer Murata -> Capacitor_SMD:C_0402_1005Metric; Part Number GRM033R61A224KE90D -> Capacitor_SMD:C_0402_1005Metric
- C4, C8: footprint Capacitor_SMD:C_0201_0603Metric -> Capacitor_SMD:C_0402_1005Metric; Manufacturer Murata -> Capacitor_SMD:C_0402_1005Metric; Part Number GRM033R61A105ME44D -> Capacitor_SMD:C_0402_1005Metric
- C6, C7: value 1 uF -> C; Manufacturer Murata -> (none); Part Number GRM033R61A105ME44D -> (none); now not fitted
- C9: value 220 nF -> 1 uF; footprint Capacitor_SMD:C_0201_0603Metric -> Capacitor_SMD:C_0402_1005Metric; Manufacturer Murata -> (none); Part Number GRM033R61A224KE90D -> (none)
- D1: footprint limiters:SMP1345-087LF -> eval:TSLP-2-19; Manufacturer Skyworks -> Infineon; Part Number SMP1345-087LF -> BAR9002ELE6327XTMA1
- D14: footprint limiters:SMP1345-087LF -> eval:TSLP-2-19; Manufacturer Skyworks -> Infineon; Part Number SMP1345-087LF -> BAR9002ELE6327XTMA1; Substitution SMP1302-087LF, SMP1331-087LF -> (none)
- D2, D38, D8: footprint Diode_SMD:D_0201_0603Metric -> eval:TSSLP-2-1
- D37, D5: footprint Diode_SMD:D_0201_0603Metric -> eval:TSLP-2-19; Part Number BAR9002ELSE6327XTSA1 -> BAR9002ELE6327XTMA1
- D4, D7: footprint Diode_SMD:D_0201_0603Metric -> eval:TSLP-2-19; Part Number BAR9002ELSE6327XTSA1 -> BAR9002ELE6327XTMA1; Substitution Toshiba JDP2S08SC -> (none)
- L1: value 33nH -> L; Manufacturer Murata -> (none); Part Number LQP03TN33NJ02D -> (none)
- L2: value 47uH -> L; footprint Inductor_SMD:L_0603_1608Metric -> Inductor_SMD:L_0201_0603Metric; Manufacturer Taiyo Yuden -> (none); Part Number LSQNB160808T470M -> (none); Substitution LSQNB160808T470K -> (none)
- L4: value 33nH -> L; footprint Inductor_SMD:L_0201_0603Metric -> Inductor_SMD:L_0805_2012Metric; Manufacturer Murata -> (none); Part Number LQP03TN33NJ02D -> (none)
- L5: value 47uH -> 1.0 nH; footprint Inductor_SMD:L_0603_1608Metric -> Inductor_SMD:L_0201_0603Metric; Manufacturer Taiyo Yuden -> Murata; Part Number LSQNB160808T470M -> LQP03HQ1N0W02D; Substitution LSQNB160808T470K -> (none)
- R12, R16: value 1k -> 10k
- R15: value 10k -> 0
- R17: value 1k -> R; footprint Resistor_SMD:R_0402_1005Metric -> Resistor_SMD:R_0201_0603Metric
- R2: value 10k -> 0; now fitted
- R40: value 1k -> 10k; now not fitted
- R41: value 10k -> 0; now not fitted
- R42: value 1k -> 0
- R5, R6: value 10k -> R; footprint Resistor_SMD:R_0402_1005Metric -> Resistor_SMD:R_0201_0603Metric; now not fitted
- R7, R8: value 1k -> R; footprint Resistor_SMD:R_0402_1005Metric -> Resistor_SMD:R_0201_0603Metric; now not fitted
Connections:
- net GND: now also C11.1, C21.2, C24.2, C32.2, C7.1, D1.2 (A), D4.1 (K), R12.2, R16.2, R41.2, R8.2, C15.2, C20.2, C27.2, C28.2, C29.2, C34.2, C35.2, D10.2 (A), D12.2 (A), D6.2 (A), J11.2 (Ext), J12.2 (Ext), J13.2 (Ext), J14.2 (Ext), J17.2 (Ext), J18.2 (Ext), J3.2 (Ext), J4.2 (Ext), J5.2 (Ext), J6.2 (Ext), Q1.1 (S), Q2.1 (S), Q4.1 (S), R22.2, R23.2, R24.2, R25.2, R27.2, R33.2, R35.2, R58.2, U1.1 (NC), U1.3 (NC), U1.4 (NC), U1.6 (NC), U1.7 (GND), U2.4 (V-); no longer C1.2, C3.2, C4.2, C6.2, C7.2, C8.2, D1.1 (K), D2.2 (A), L2.2, L5.2, R1.2, R40.2, R5.2
- net VCC: now also R17.2, R5.2, R7.1, C28.1, C34.1, C35.1, L7.2, Q1.4 (S), Q2.4 (S), Q4.4 (S), R34.1, R57.1, U2.8 (V+); no longer C3.1, C4.1, C6.1, C7.1, C8.1, R15.1, R2.2, R41.2, R6.1
- net at J15.1 (In): now also C30.1; no longer C17.2
- net at C18.1: now also D3.1 (K), L6.2
- net at C18.2: now also J12.1 (In); no longer L4.1
- net at C17.1: now also J11.1 (In)
- net at C11.2: now also R3.2
- net at C12.1: now also J6.1 (In); no longer J10.1 (In)
- net at D14.2 (A): now also C31.1, C33.2, D12.1 (K), D13.2 (A); no longer C23.1
- net at C23.2: now also C24.1, R29.1, R32.2, R33.1, R34.2, U2.3 (+)
- net at C22.1: now also C23.1, R30.1, R32.1, R55.2, R56.2, U2.1
- net at C22.2: now also R28.1, R30.2, R35.1, U2.2 (-); no longer D2.1 (K)
- net at C21.1: now also R40.1, C25.1, C26.1, D3.2 (A), R27.1, R31.1, U2.7
- net at C31.2: now also J17.1 (In)
- net at C32.1: now also R13.1, R14.1, R15.1, D13.1 (K)
- net at C67.1: now also C70.2, D5.2 (A), L1.1; no longer D5.1 (K)
- net at R12.1: now also J16.1 (Pin_1), J16.2 (Pin_2), Q1.2 (G), Q1.5 (G)
- net at R41.1: now also C25.2, R31.2, R55.1, U2.6 (-); no longer R40.1
- net at R11.1: now also R10.1, R9.1, C29.1, D11.1 (K)
- net at L4.2: now also R17.1, R21.2, R3.1; no longer L5.1
- net at C71.1, R42.1, R43.1: now also D5.1 (K); no longer D5.2 (A)
- net at L1.2, L2.1: now also R4.1
- net at R1.1, R2.1: now also D2.1 (K), C15.1, R24.1; no longer C1.1, D4.2 (A)
- net at C63.1, D37.1 (K): now also C69.2, D38.2 (A), L9.1
- net at R7.2: now also C7.2; no longer R5.1
- net at R10.2: now also Q1.3 (D); no longer R12.2
- net at R8.1: now also C6.1; no longer R6.2
- net at R14.2: now also Q2.3 (D)
- net at R16.1: now also J19.1 (Pin_1), J19.2 (Pin_2), Q2.2 (G), Q2.5 (G); no longer R15.2
- new net: J9.1 (Pin_1), J9.2 (Pin_2), Q4.2 (G), Q4.5 (G), R23.1
- new net: Q4.6 (D), R2.2
- new net: C14.2, L2.2, L4.1, R21.1, R4.2
- new net: C12.2, D2.2 (A), L5.1
- new net: Q4.3 (D), R1.2
- new net: C30.2, C8.1, D10.1 (K), D11.2 (A)
- new net: C20.1, D9.1 (K), R25.1, R28.2, R29.2
- new net: C33.1, J18.1 (In)
- new net: C14.1, R22.1
- new net: C26.2, C27.1, R40.2, R56.1, R57.2, R58.1, U2.5 (+)
- new net: Q2.6 (D), R15.2
- new net: C8.2, J14.1 (In)
- new net: C16.1, C17.2, D4.2 (A), D6.1 (K)
- new net: Q1.6 (D), R11.2
- new net: C6.2, L7.1, L8.2, R5.1, R6.2
- new net: C1.1, U1.2 (RFIN)
- new net: C3.2, U1.5 (RFOUT)
- new net: C3.1, J4.1 (In)
- new net: C19.1, J13.1 (In)
- new net: C19.2, D9.2 (A), L6.1
- new net: L8.1, L9.2, R6.1
- new net: C4.1, D1.1 (K), L5.2
- new net: C1.2, J3.1 (In)
- new net: C16.2, J10.1 (In)
- new net: C4.2, J5.1 (In)
Other:
- note added: "Switched PIN-Schottky"
- note removed: "PIN"
- note removed: "PIN-PIN"
- moved on the sheet: C10, C13, C63, C64, C67, C68, C69, C70, C9, D37, D38, D5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
