File: evaluation-boards/filters/filters.kicad_sch (KiCad schematic)
At the start: 63 parts, among them J1 Conn_Coaxial, J10 Conn_Coaxial, J11 Conn_Coaxial, J12 Conn_Coaxial, J13 Conn_Coaxial, J14 Conn_Coaxial, J15 Conn_Coaxial, J16 Conn_Coaxial, J17 Conn_Coaxial, J18 Conn_Coaxial, J19 Conn_Coaxial, J2 Conn_Coaxial, J20 Conn_Coaxial, J3 Conn_Coaxial, J4 Conn_Coaxial, J5 Conn_Coaxial, J6 Conn_Coaxial, J7 Conn_Coaxial, J8 Conn_Coaxial, J9 Conn_Coaxial, U1 FIL-DEA, U3 FIL-LP0603, U5 5130BP18U4060, U7 2450HP

Commit message: Update filters board
Parts:
- removed C15, C16, C19, C20, C5: C, Capacitor_SMD:C_0201_0603Metric, symbol Device:C
- removed L16, L4, L7: L, Inductor_SMD:L_0201_0603Metric, symbol Device:L
- removed U1: FIL-DEA, gsg-modules:FIL-DEA-0603, symbol gsg-symbols:FIL-DEA
- removed U3: FIL-LP0603, gsg-modules:LP0603, symbol gsg-symbols:FIL-LP0603
- removed U5: 5130BP18U4060, gsg-modules:5130BP18U4060, symbol gsg-symbols:5130BP18U4060
- removed U7: 2450HP, gsg-modules:2500BL14M100, symbol gsg-symbols:2450HP
- added C8: C, Capacitor_SMD:C_0201_0603Metric, symbol Device:C
- added FL1: BPF, eval:Filter_Pulse_BPF1608LM09R5000A, symbol RF_Filter:BFCN-1445
- added FL2: B39162B8813P810, Filter:Filter_1109-5_1.1x0.9mm, symbol Filter:B39162B8813P810
- added L8: L, Inductor_SMD:L_0201_0603Metric, symbol Device:L
- added R4: 100, Resistor_SMD:R_0201_0603Metric, symbol Device:R
- R1, R2, R3: value R -> 100
- renumbered C8 to C5, L8 to L4
Connections:
- net GND: now also C12.1, C13.1, C14.1, C17.1, C18.1, C5.1, C6.1, C7.1, R1.2, R2.2, FL1.2 (GND), FL1.4 (GND), FL2.2, FL2.3, FL2.5, L8.2, R4.2; no longer L13.2, L14.2, L15.2, L4.2, L5.2, L6.2, R1.1
- net at J8.1 (In): now also J7.1 (In)
- net at J9.1 (In): now also C1.1
- net at J10.1 (In): now also C4.2
- net at J11.1 (In): now also C8.1
- net at J12.1 (In): now also C11.2
- net at J14.1 (In): now also C17.2, L6.2
- net at J13.1 (In): now also C5.2, L4.1
- net at J4.1 (In): now also R1.1, R2.1
- net at J16.1 (In): now also C18.2, L15.2
- net at C9.1: now also L10.1, C8.2; no longer C5.2
- net at J18.1 (In): now also L9.1, FL2.4
- net at L15.1: now also C14.2, L14.2; no longer C18.2
- net at L12.1: now also C10.2, C11.1; no longer C14.2
- net at J3.1 (In): now also R3.1, R4.1; no longer C1.1
- net at L13.1: now also C12.2, J15.1 (In); no longer C17.1
- net at C6.2, L5.1: now also L4.2; no longer C7.1
- net at C7.2, L6.1: now also L5.2; no longer C5.1
- net at C10.1, C9.2: now also L11.1; no longer L4.1
- net at J17.1 (In): now also FL2.1, L8.1
- net at J5.1 (In): no longer C6.1
- net at J6.1 (In): no longer C10.2
- new net: FL1.1 (IN), J20.1 (In)
- new net: FL1.3 (OUT), J19.1 (In)
- new net: C13.2, L13.2, L14.1
- no-connect marks 0 -> 2
Other:
- moved on the sheet: C1, C2, C3, C4, C5, C6, C7, J1, J2, J3, J4, J5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

Commit message: Update filters board
Parts:
- removed C1, C10, C11, C12, C13, C14, C17, C18, C2, C3, C4, C5, C6, C7, C8, C9: C, Capacitor_SMD:C_0201_0603Metric, symbol Device:C
- removed FL2: B39162B8813P810, Filter:Filter_1109-5_1.1x0.9mm, symbol Filter:B39162B8813P810
- removed L1, L10, L11, L12, L13, L14, L15, L2, L3, L4, L5, L6, L8, L9: L, Inductor_SMD:L_0201_0603Metric, symbol Device:L
- added FL2, FL3, FL4, FL5, FL6: BPF, eval:Filter_Pulse_BPF1608LM09R5000A, symbol RF_Filter:BFCN-1445
- added TP1, TP2: TestPoint, eval:Square_Pad_0.364x0.364mm, symbol Connector:TestPoint
- J1, J10, J11, J12, J13, J14, J15, J16, J17, J18, J19, J2, J20, J3, J4, J5, J6, J7, J8, J9: footprint sma-variants:Linx_SMA_CONSMA003.062 -> eval:SMA_MyAntenna_A-SMA-KE-16.5A_EdgeMount
Connections:
- net GND: now also FL2.2 (GND), FL2.4 (GND), FL3.2 (GND), FL3.4 (GND), FL4.2 (GND), FL4.4 (GND), FL5.2 (GND), FL5.4 (GND), FL6.2 (GND), FL6.4 (GND)
- net at J17.1 (In): now also FL2.3 (OUT)
- net at J16.1 (In): now also FL3.1 (IN)
- net at J14.1 (In): now also FL4.1 (IN)
- net at J11.1 (In): now also FL5.3 (OUT)
- net at J12.1 (In): now also FL5.1 (IN)
- net at J18.1 (In): now also FL2.1 (IN)
- net at J10.1 (In): now also FL6.1 (IN)
- net at J15.1 (In): now also FL3.3 (OUT)
- net at J9.1 (In): now also FL6.3 (OUT)
- net at J13.1 (In): now also FL4.3 (OUT)
- net at J5.1 (In): now also TP1.1
- net at J6.1 (In): now also TP2.1
- no-connect marks 2 -> 0
Other:
- moved on the sheet: J10, J12, J14, J16, J18
