File: evaluation-boards/baluns/baluns.kicad_sch (KiCad schematic)
At the start: 182 parts, among them J1 CONN_COAXIAL, J10 CONN_COAXIAL, J11 CONN_COAXIAL, J12 CONN_COAXIAL, J13 CONN_COAXIAL, J14 CONN_COAXIAL, J15 CONN_COAXIAL, J16 CONN_COAXIAL, J17 CONN_COAXIAL, J18 CONN_COAXIAL, J2 CONN_COAXIAL, J3 CONN_COAXIAL, J4 CONN_COAXIAL, J5 CONN_COAXIAL, J6 CONN_COAXIAL, J7 CONN_COAXIAL, J8 CONN_COAXIAL, J9 CONN_COAXIAL, P1 Conn_01x02, P2 Conn_01x02, P3 Conn_01x02, P4 Conn_01x02, P5 Conn_01x02, Q1 BFR840, Q2 BFR840, Q3 BFR840, Q4 BFR840, Q5 BFP840ESD, Q6 BFP840ESD, Q7 BFP840ESD, Q8 BFP840ESD, T1 B0310J50100AHF, T2 B0310J50100AHF

Commit message: Update baluns board
Parts:
- removed C10, C11, C12, C13, C17, C19, C20, C21, C22, C23, C24, C26, C27, C29, C31, C32, C35, C36, C37, C38, C39, C40, C44, C45, C47, C48, C7, C8, C9: 1 uF, Capacitor_SMD:C_0201_0603Metric, symbol Device:C
- removed C14, C15, C16, C18, C30, C33, C34, C43: 0.3 pF, Capacitor_SMD:C_0201_0603Metric, symbol Device:C
- removed J12, J13, J14, J15, J16, J17, J18: CONN_COAXIAL, sma-variants:SMA-EDGE-1.3mm-pad-1.05mm-gap-2.6mm-keepout, symbol Connector:Conn_Coaxial
- removed L10: 18 nH, Inductor_SMD:L_0201_0603Metric, symbol Device:L
- removed L11: L, Inductor_SMD:L_0805_2012Metric, symbol Device:L
- removed L12, L9: L, Inductor_SMD:L_0201_0603Metric, symbol Device:L
- removed L14: 5.6 nH, Inductor_SMD:L_0201_0603Metric, symbol Device:L
- removed Q1, Q2, Q3, Q4: BFR840, eval:TSLP-3-9, symbol Transistor_BJT:Q_NPN_BCE
- removed Q5, Q6, Q7, Q8: BFP840ESD, eval:SOT-343-4-3, symbol eval:Q_NPN_BECE
- removed R10, R24, R46, R59, R71, R77, R79, R8, R80, R83: 220, Resistor_SMD:R_0201_0603Metric, symbol Device:R
- removed R11, R13, R19, R20, R26, R27, R29, R30, R31, R32, R33, R34, R36, R42, R47, R48, R49, R50, R51, R52, R55, R56, R57, R60, R61, R62, R65, R69, R72, R78, R81, R84, R85, R86: 0, Resistor_SMD:R_0201_0603Metric, symbol Device:R
- removed R14, R21, R37, R43, R6, R63, R73: 4.3k, Resistor_SMD:R_0201_0603Metric, symbol Device:R
- removed R15, R22, R38, R44, R64, R74, R9: 2.4k, Resistor_SMD:R_0201_0603Metric, symbol Device:R
- removed R16, R39, R66: 300, Resistor_SMD:R_0201_0603Metric, symbol Device:R
- removed R17, R40, R70: 200, Resistor_SMD:R_0201_0603Metric, symbol Device:R
- removed R18, R75, R82: 6.8k, Resistor_SMD:R_0201_0603Metric, symbol Device:R
- removed R23, R45, R7, R76: 470, Resistor_SMD:R_0201_0603Metric, symbol Device:R
- removed R25, R53: 43, Resistor_SMD:R_0201_0603Metric, symbol Device:R
- removed R28, R41, R54, R58, R67, R68: 82, Resistor_SMD:R_0201_0603Metric, symbol Device:R
- removed T1: B0310J50100AHF, RF_Converter:Anaren_0805_2012Metric-6, symbol eval:B0310J50100AHF
- added C112, C203: 8p2, Capacitor_SMD:C_0201_0603Metric, symbol Device:C
- added C171, C207, C208, C210, C211, C212, C213, C214, C215: 1 uF, Capacitor_SMD:C_0201_0603Metric, symbol Device:C
- added C202: 2.2nF, Capacitor_SMD:C_0201_0603Metric, symbol Device:C
- added D10: Schottky, eval:TSLP-2-19, symbol Device:D_Schottky
- added L19: 47uH, eval:L_Taiyo-Yuden_A251818, symbol Device:L
- added L20: 33 nH, Inductor_SMD:L_0201_0603Metric, symbol Device:L
- added L29: 100uH, eval:L_TDK_MLZ2012_h1.25mm, symbol Device:L
- added L30: 56 nH, Inductor_SMD:L_0201_0603Metric, symbol Device:L
- added Q15, Q17: BFR840, eval:TSLP-3-9, symbol Transistor_BJT:Q_NPN_BCE
- added Q16, Q18: Q_PMOS_GSD, eval:TSLP-3-9, symbol Transistor_FET:Q_PMOS_GSD
- added R142, R143, R144, R162, R163, R171, R172: 0, Resistor_SMD:R_0201_0603Metric, symbol Device:R
- added R147, R155, R158, R159, R166, R168: 100, Resistor_SMD:R_0201_0603Metric, symbol Device:R
- added R152: 330, Resistor_SMD:R_0201_0603Metric, symbol Device:R
- added R153, R165: 120, Resistor_SMD:R_0201_0603Metric, symbol Device:R
- added R154: 33k, Resistor_SMD:R_0201_0603Metric, symbol Device:R
- added R156, R173: 220, Resistor_SMD:R_0201_0603Metric, symbol Device:R
- added R157: 750, Resistor_SMD:R_0201_0603Metric, symbol Device:R
- added R160: 51, Resistor_SMD:R_0201_0603Metric, symbol Device:R
- added R161, R169, R170: 10, Resistor_SMD:R_0201_0603Metric, symbol Device:R
- added R164: 3.3k, Resistor_SMD:R_0201_0603Metric, symbol Device:R
- added R167: 4k7, Resistor_SMD:R_0201_0603Metric, symbol Device:R
- C1, C2, C5, C6: value 0.3 pF -> 1 uF; Manufacturer (none) -> Murata; Part Number (none) -> GRM033R61A105ME44D; Substitution (none) -> GRM033R61A105ME44*, GRM033R61C105ME15*, Samsung CL03A105MO3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; now fitted
- C25: Manufacturer (none) -> Murata; Part Number (none) -> GRM033R61A105ME44D; Substitution (none) -> GRM033R61A105ME44*, GRM033R61C105ME15*, Samsung CL03A105MO3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; now fitted
- C28, C41, C42, C46, C49: Manufacturer (none) -> Murata; Part Number (none) -> GRM033R61A105ME44D; Substitution (none) -> GRM033R61A105ME44*, GRM033R61C105ME15*, Samsung CL03A105MO3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
- C3: value 0.3 pF -> 8p2; Manufacturer (none) -> Murata; Part Number (none) -> GRM0335C1H8R2CA01D; Substitution (none) -> GRM0335C1H8R2*; now fitted
- C4: value 0.3 pF -> 2.2nF; Manufacturer (none) -> Murata; Part Number (none) -> GRM033R71A222KA01D; Substitution (none) -> GRM033R71A222KA01*; now fitted
- J1, J10, J11, J2, J3, J4, J5, J6, J7, J8, J9: footprint sma-variants:SMA-EDGE-1.3mm-pad-1.05mm-gap-2.6mm-keepout -> eval:SMA_MyAntenna_A-SMA-KE-16.5A_EdgeMount
- L1: value 18 nH -> DNP
- L13: value L -> 62nH; footprint Inductor_SMD:L_0805_2012Metric -> Inductor_SMD:L_0603_1608Metric; Manufacturer (none) -> Murata; Part Number (none) -> LQW18AN62NJ00D; Substitution (none) -> LQW18AN62N*
- L2: value 5.6 nH -> 100uH; footprint Inductor_SMD:L_0201_0603Metric -> eval:L_TDK_MLZ2012_h1.25mm; Manufacturer (none) -> TDK; Part Number (none) -> MLZ2012N101LT000; Substitution (none) -> MLZ2012N101LTD25
- L3: value 18 nH -> 56 nH; Manufacturer (none) -> Murata; Part Number (none) -> LQP03TN56NJ02D; Substitution (none) -> LQP03TN56NH02D
- L4: value 5.6 nH -> 2.4 nH; Manufacturer (none) -> Murata; Part Number (none) -> LQP03TN2N4C02D; Substitution (none) -> LQP03TN2N4B02D
- L5: value 18 nH -> 100uH; footprint Inductor_SMD:L_0201_0603Metric -> eval:L_TDK_MLZ2012_h1.25mm; Manufacturer (none) -> TDK; Part Number (none) -> MLZ2012N101LT000; Substitution (none) -> MLZ2012N101LTD25; now fitted
- L6: value 5.6 nH -> 56 nH; Manufacturer (none) -> Murata; Part Number (none) -> LQP03TN56NJ02D; Substitution (none) -> LQP03TN56NH02D
- L7: value L -> 100uH; footprint Inductor_SMD:L_0201_0603Metric -> eval:L_TDK_MLZ2012_h1.25mm; Manufacturer (none) -> TDK; Part Number (none) -> MLZ2012N101LT000; Substitution (none) -> MLZ2012N101LTD25
- L8: value L -> 56 nH; footprint Inductor_SMD:L_0805_2012Metric -> Inductor_SMD:L_0201_0603Metric; Manufacturer (none) -> Murata; Part Number (none) -> LQP03TN56NJ02D; Substitution (none) -> LQP03TN56NH02D
- R1: value 82 -> 33k; Manufacturer (none) -> Yageo; Part Number (none) -> RC0201JR-0733KL; Substitution (none) -> any equivalent
- R12: value 0 -> 220; Manufacturer (none) -> Yageo; Part Number (none) -> RC0201JR-07220RL; Substitution (none) -> any equivalent; now fitted
- R2: value 2.4k -> 0; Manufacturer (none) -> Yageo; Part Number (none) -> RC0201JR-070RL; Substitution (none) -> any equivalent; now fitted
- R3: value 4.3k -> 51; Manufacturer (none) -> Yageo; Part Number (none) -> RC0201JR-0751RL; Substitution (none) -> any equivalent; now fitted
- R35: value 82 -> 220; Manufacturer (none) -> Yageo; Part Number (none) -> RC0201JR-07220RL; Substitution (none) -> any equivalent
- R4: value 300 -> 100; Manufacturer (none) -> Yageo; Part Number (none) -> RC0201JR-07100RL; Substitution (none) -> any equivalent; now fitted
- R5: value 200 -> 10; Manufacturer (none) -> Yageo; Part Number (none) -> RC0201JR-0710RL; Substitution (none) -> any equivalent; now fitted
- T2: value B0310J50100AHF -> RF_BALUN; Manufacturer (none) -> TTM; Part Number (none) -> B0310J50100AHF
Connections:
- net GND: now also C41.2, C42.2, C5.1, P3.2 (Pin_2), P4.2 (Pin_2), R4.2, C171.2, C211.2, C212.2, C214.2, C215.2, R143.1, R147.2, R152.1, R158.2, R159.2, R164.2, R166.2, R168.2; no longer C3.2, C4.2, C42.1, C5.2, C6.2, R1.1, R35.1
- net at J2.1 (In): now also L1.1, C213.1; no longer C2.1
- net at J1.1 (In): now also C28.2; no longer C3.1
- net VAA: now reaches P2.1 (Pin_1), P2.2 (Pin_2)
- net VAA: now also C1.1, C2.1, C41.1, C42.1, L2.1, L5.1, L7.1, P5.1 (Pin_1), R1.1, C214.1, C215.1, L29.1, Q16.3 (D), Q18.3 (D), R154.1
- net at L13.2: now also J10.1 (In), J11.1 (In), L20.2
- net at P5.2 (Pin_2): now also C171.1, D10.2 (A); no longer P5.1 (Pin_1)
- net at L7.2, L8.1: now also C4.2, R5.1
- net at T2.4: now also J8.1 (In), L6.2, R3.2; no longer L7.1
- net at L1.2: now also J3.1 (In), C208.1
- net at L4.1: now also Q17.2 (C), R172.2, R173.2
- net at T2.3: now also J7.1 (In), L8.2, R5.2
- net at P4.1 (Pin_1): now also R1.2, Q18.1 (G); no longer P4.2 (Pin_2)
- net at J9.1 (In): now also C6.1
- net at P3.1 (Pin_1): now also Q16.1 (G), R154.2; no longer P3.2 (Pin_2)
- net at C49.2: now also J4.1 (In), L3.2, R144.2
- net at R12.2: now also L13.1, C112.2, L19.2
- net at R35.2: now also C112.1; no longer R1.2
- net at C25.2: now also R153.1
- net at L4.2: now also C207.1
- net at L2.2: now also L3.1, C202.2, R144.1
- net at J6.1 (In): now also C46.2; no longer C28.1
- net at C25.1: now also R155.2
- net at T2.1: now also C6.2
- net at R12.1: now also L20.1
- net at C49.1: now also R169.1; no longer L13.1
- net at C46.1: now also R172.1
- net at L6.1: now also C3.1, L5.2, R3.1
- net at R2.2: now also C3.2; no longer R3.1
- net at C4.1: now also R4.1
- net at T2.2 (GND): now also C5.2
- net at J5.1 (In): now also C210.2, L30.2, R142.2
- new net: Q16.2 (S), R163.1
- new net: C212.1, R156.2, R157.1, R163.2
- new net: C211.1, R167.1, R171.2, R173.1
- new net: Q17.1 (B), R164.1, R165.2, R167.2, R170.2
- new net: C203.1, L29.2, L30.1, R142.1
- new net: Q17.3 (E), R166.1, R168.1, R169.2
- new net: Q15.3 (E), R158.1, R159.1, R161.1
- new net: C210.1, R170.1
- new net: C207.2, R165.1
- new net: Q18.2 (S), R171.1
- new net: C203.2, R143.2
- new net: Q15.1 (B), R152.2, R153.2, R157.2, R162.1
- new net: C202.1, R147.1
- new net: C28.1, R162.2
- new net: C213.2, R161.2
- new net: D10.1 (K), L19.1, R35.1
- new net: Q15.2 (C), R155.1, R156.1, R160.1
- new net: C208.2, R160.2
Other:
- moved on the sheet: J1, J10, J11, J2, J3, J4, J5, J6, J7, J8, J9, P1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
