File: evaluation-boards/rf-amps/rf-amps.kicad_pcb (KiCad board)
At the start: 4 copper layers, 23 x 100 mm, 126 parts, among them J1 CONN_COAXIAL, J10 CONN_COAXIAL, J11 CONN_COAXIAL, J12 CONN_COAXIAL, J13 CONN_COAXIAL, J14 CONN_COAXIAL, J2 CONN_COAXIAL, J3 CONN_COAXIAL, J4 CONN_COAXIAL, J5 CONN_COAXIAL, J6 CONN_COAXIAL, J7 CONN_COAXIAL, J8 CONN_COAXIAL, J9 CONN_COAXIAL, P1 Conn_01x02, P2 Conn_01x02, P3 CONN_02X03, P4 CONN_02X03, P5 CONN_01X03, P6 CONN_01X03, P7 CONN_01X03, P8 CONN_01X03, P9 CONN_01X03, Q1 BFR840, Q2 BFR840, Q3 BFP840ESD, Q4 BFP840ESD, U1 BGA9H1BN6, U2 BGA8U1BN6, U3 BGB741L7ESD

Commit message: Update rf-amps board
Parts:
- removed C1, C2, C27, C33, C5, C7, C8, C9: 1uF, Capacitor_SMD:C_0201_0603Metric
- removed C26, C4, C40, C41, C43, C44, C49, C50, C6: C, Capacitor_SMD:C_0201_0603Metric
- removed C28, C34, C48: 39pF, Capacitor_SMD:C_0201_0603Metric
- removed C29, C35: 3.3pF, Capacitor_SMD:C_0201_0603Metric
- removed C30, C36: 1pF, Capacitor_SMD:C_0201_0603Metric
- removed C31, C32, C37, C38: 10pF, Capacitor_SMD:C_0201_0603Metric
- removed L12, L13: 5.1nH, Inductor_SMD:L_0201_0603Metric
- removed L17, L19: 47uH, Inductor_SMD:L_0603_1608Metric
- removed L18, L20: 33nH, Inductor_SMD:L_0201_0603Metric
- removed L25, L26, L27, L8: L, Inductor_SMD:L_0201_0603Metric
- removed L3: 4.7 nH, Inductor_SMD:L_0201_0603Metric
- removed P9: CONN_01X03, Connector_PinHeader_2.54mm:PinHeader_1x03_P2.54mm_Vertical
- removed Q3, Q4: BFP840ESD, eval:SOT-343-4-3
- removed R1, R14, R15, R24, R26, R40, R45, R46, R47, R48: 0, Resistor_SMD:R_0201_0603Metric
- removed R11, R25: R, Resistor_SMD:R_0201_0603Metric
- removed R12: 33k, Resistor_SMD:R_0201_0603Metric
- removed R13: 27, Resistor_SMD:R_0201_0603Metric
- removed R16, R21: 30k, Resistor_SMD:R_0201_0603Metric
- removed R17, R18, R22: 82, Resistor_SMD:R_0201_0603Metric
- removed R20, R23: 10, Resistor_SMD:R_0201_0603Metric
- added C11: 1 uF, Capacitor_SMD:C_0201_0603Metric, F.Cu at (140.4, 78.5)
- added C12: 1 uF, Capacitor_SMD:C_0201_0603Metric, F.Cu at (140.4, 90.5)
- added C15: 220 nF, Capacitor_SMD:C_0201_0603Metric, F.Cu at (138.3, 80.0)
- added C39: 220 nF, Capacitor_SMD:C_0201_0603Metric, F.Cu at (144.8, 80.3)
- added C42: 220 nF, Capacitor_SMD:C_0201_0603Metric, F.Cu at (137.6, 92.0)
- added C51: 220 nF, Capacitor_SMD:C_0201_0603Metric, F.Cu at (144.8, 92.3)
- added C57: 1 uF, Capacitor_SMD:C_0201_0603Metric, F.Cu at (139.4, 78.3)
- added C58: 1 uF, Capacitor_SMD:C_0201_0603Metric, F.Cu at (141.6, 80.8)
- added C59: 1 uF, Capacitor_SMD:C_0201_0603Metric, F.Cu at (140.2, 81.5)
- added C60: 1 uF, Capacitor_SMD:C_0201_0603Metric, F.Cu at (137.9, 90.2)
- added C61: 1 uF, Capacitor_SMD:C_0201_0603Metric, F.Cu at (141.6, 92.8)
- added C62: 1 uF, Capacitor_SMD:C_0201_0603Metric, F.Cu at (140.2, 93.5)
- added L14: 1.8 nH, Inductor_SMD:L_0201_0603Metric, F.Cu at (142.6, 128.3)
- added L28: 15 uH, Inductor_SMD:L_0603_1608Metric, F.Cu at (143.0, 80.7)
- added L29: 15 uH, Inductor_SMD:L_0603_1608Metric, F.Cu at (143.0, 92.7)
- added L30: 15 uH, Inductor_SMD:L_0603_1608Metric, F.Cu at (139.0, 90.9)
- added L31: 15 uH, Inductor_SMD:L_0603_1608Metric, F.Cu at (141.5, 143.2)
- added L32: L, Inductor_SMD:L_0805_2012Metric, F.Cu at (141.5, 152.0)
- added R10: 470, Resistor_SMD:R_0201_0603Metric, F.Cu at (139.4, 103.7)
- added R27: 2.2k, Resistor_SMD:R_0201_0603Metric, F.Cu at (141.9, 78.1)
- added R29: 2.2k, Resistor_SMD:R_0201_0603Metric, F.Cu at (141.9, 90.1)
- added R42: 360, Resistor_SMD:R_0201_0603Metric, F.Cu at (140.2, 80.8)
- added R43: 360, Resistor_SMD:R_0201_0603Metric, F.Cu at (140.2, 92.8)
- added R44: 0, Resistor_SMD:R_0201_0603Metric, F.Cu at (141.6, 81.5)
- added R49: 0, Resistor_SMD:R_0201_0603Metric, F.Cu at (144.1, 80.3)
- added R50: 0, Resistor_SMD:R_0201_0603Metric, F.Cu at (141.6, 93.5)
- added R51: 0, Resistor_SMD:R_0201_0603Metric, F.Cu at (144.1, 92.3)
- added R52: 3, Resistor_SMD:R_0201_0603Metric, F.Cu at (143.2, 116.3)
- added R53: 3, Resistor_SMD:R_0201_0603Metric, F.Cu at (143.2, 128.3)
- added R54: 0, Resistor_SMD:R_0201_0603Metric, F.Cu at (139.7, 143.2)
- added R55: 0, Resistor_SMD:R_0201_0603Metric, F.Cu at (143.2, 141.4)
- added U4: SMA3109, Package_TO_SOT_SMD:SOT-363_SC-70-6, F.Cu at (141.5, 140.9)
- C10, C17, C55: value 1uF -> 1 uF
- C14, C16, C21: value 1uF -> 220 nF
- C18: value 1pF -> 1 uF
- C19, C24: value 18pF -> 220 nF
- C20, C22: value 22pF -> 220 nF
- C23: value 1pF -> 220 nF
- C25, C53, C56: value C -> 1 uF
- C45, C46: value 39pF -> 220 nF
- C47: value 39pF -> C
- J1, J10, J11, J12, J13, J14, J2, J3, J4, J5, J6, J7, J8, J9: footprint sma-variants:Linx_SMA_CONSMA003.062 -> sma-variants:SMA-EDGE-1.3mm-pad-1.05mm-gap-2.6mm-keepout
- L10: value 3.7nH -> 1.8 nH
- L11: value 2.2nH -> L
- P3, P4: value CONN_02X03 -> CONN_01X03; footprint Connector_PinHeader_2.54mm:PinHeader_2x03_P2.54mm_Vertical -> Connector_PinHeader_2.54mm:PinHeader_1x03_P2.54mm_Vertical
- R19: value 0 -> 470
- R2: value R -> 2.2k
- R3: value 33k -> 4900
- R36: value R -> 360
- R4, R7: value 120 -> 330
- R5: value 27 -> 220
- R6: value 0 -> 4900
- R8: value 0 -> 220
- R9: value 82 -> R
- U1: value BGA9H1BN6 -> BGB741L7ESD; footprint eval:TSLP-6-4_1.1x0.7mm_P0.4mm -> rf-amps:TSLP-7-1
- U2: value BGA8U1BN6 -> BGB741L7ESD; footprint eval:TSLP-6-4_1.1x0.7mm_P0.4mm -> rf-amps:TSLP-7-1
- moved C25 27.2 mm to (139.7, 141.8), turned to 90 degrees
- moved R6 16.5 mm to (140.4, 127.0), turned to 90 degrees
- moved C23 14.5 mm to (140.1, 138.9), turned to 180 degrees
- moved C24 13.4 mm to (143.9, 141.4), turned to -90 degrees
- moved C18 11.9 mm to (142.9, 126.6)
- moved C55 9.55 mm to (139.2, 106.2), turned to 0 degrees
- moved R38 9.08 mm to (139.2, 107.0), turned to 180 degrees
- moved R4 6.68 mm to (141.5, 116.7), turned to 0 degrees
- moved L23 5.80 mm to (141.4, 106.5), turned to 180 degrees
- moved C17 5.70 mm to (142.9, 114.6), turned to 180 degrees
- moved R37 5.28 mm to (140.8, 105.5), turned to 180 degrees
- moved C22 5.01 mm to (143.9, 128.3), turned to -90 degrees
- moved R7 4.91 mm to (141.5, 128.7)
- moved R9 4.66 mm to (142.9, 138.9), turned to 0 degrees
- moved C45 4.50 mm to (140.4, 116.3), turned to 90 degrees
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Connections:
- C18 pad 1: GND -> Net-(P7-Pin_2)
- C18 pad 2: Net-(C18-Pad2) -> GND
- C19 pad 2: Net-(Q1-C) -> Net-(C19-Pad2)
- C21 pad 1: Net-(P7-Pin_2) -> Net-(Q2-B)
- C21 pad 2: GND -> Net-(J9-In)
- C22 pad 1: Net-(Q2-B) -> Net-(J10-In)
- C22 pad 2: Net-(J9-In) -> Net-(C22-Pad2)
- C23 pad 1: GND -> Net-(C23-Pad1)
- C23 pad 2: Net-(C23-Pad2) -> Net-(J11-In)
- C24 pad 1: Net-(J10-In) -> Net-(J12-In)
- C25 pad 1: GND -> Net-(P8-Pin_2)
- C25 pad 2: Net-(C25-Pad2) -> GND
- C45 pad 2: GND -> Net-(Q1-B)
- C46 pad 2: GND -> Net-(Q2-B)
- C47 pad 2: GND -> Net-(C23-Pad1)
- L10 pad 1: Net-(C18-Pad2) -> Net-(L10-Pad1)
- L11 pad 1: Net-(C30-Pad2) -> Net-(L11-Pad1)
- P3 pad 2: VCC -> Net-(P3-Pin_2)
- P3 pad 3: Net-(P3-Pin_3) -> GND
- P4 pad 2: VCC -> Net-(P4-Pin_2)
- P4 pad 3: Net-(P4-Pin_3) -> GND
- Q2 pad 3: Net-(Q2-E) -> GND
- R19 pad 1: Net-(P3-Pin_3) -> Net-(U1-RFIN)
- R19 pad 2: Net-(U1-C2) -> Net-(U1-BIAS)
- R3 pad 1: Net-(C25-Pad2) -> Net-(Q1-B)
- R3 pad 2: Net-(Q1-B) -> Net-(Q1-C)
- R4 pad 1: Net-(P6-Pin_2) -> Net-(C45-Pad1)
- R4 pad 2: Net-(C45-Pad1) -> Net-(L10-Pad1)
- R5 pad 1: Net-(C45-Pad1) -> Net-(Q1-C)
- R5 pad 2: Net-(C18-Pad2) -> Net-(P6-Pin_2)
- R6 pad 1: Net-(C45-Pad1) -> Net-(Q2-B)
- R6 pad 2: Net-(C25-Pad2) -> Net-(Q2-C)
- R7 pad 1: Net-(P7-Pin_2) -> Net-(C46-Pad1)
- R7 pad 2: Net-(C46-Pad1) -> Net-(L14-Pad1)
- R8 pad 1: Net-(C46-Pad1) -> Net-(Q2-C)
- R8 pad 2: Net-(C26-Pad2) -> Net-(P7-Pin_2)
- R9 pad 1: Net-(P8-Pin_2) -> Net-(C47-Pad1)
- R9 pad 2: Net-(C47-Pad1) -> Net-(L11-Pad1)
- U1 pad 1: GND -> VCC
- U1 pad 2: VCC -> Net-(U1-BIAS)
- U1 pad 3: Net-(C2-Pad2) -> Net-(U1-RFIN)
- U1 pad 4: Net-(U1-C2) -> Net-(U1-RFOUT)
- U1 pad 5: Net-(L3-Pad2) -> Net-(P3-Pin_2)
- U1 pad 6: Net-(P3-Pin_4) -> Net-(U1-ADJ)
- U2 pad 1: Net-(P4-Pin_3) -> VCC
- U2 pad 2: VCC -> Net-(U2-BIAS)
- U2 pad 4: Net-(P4-Pin_4) -> Net-(U2-RFOUT)
- U2 pad 5: GND -> Net-(P4-Pin_2)
Routing:
- net Net-(P9-Pin_2): track 20.0 -> 0.00 mm, vias 2 -> 0
- net Net-(P3-Pin_4): track 15.7 -> 0.00 mm, vias 1 -> 0
- net GND: track 26.8 -> 14.0 mm, vias 49 -> 51
- net Net-(P3-Pin_2): track 0.00 -> 11.1 mm
- net Net-(P4-Pin_2): track 0.00 -> 11.0 mm
- net Net-(P4-Pin_4): track 9.95 -> 0.00 mm
- net Net-(P3-Pin_3): track 9.32 -> 0.00 mm
- net Net-(P4-Pin_3): track 6.20 -> 0.00 mm, vias 1 -> 0
- net Net-(C25-Pad2): track 5.70 -> 0.00 mm
- net Net-(P7-Pin_2): track 16.7 -> 11.2 mm
- net Net-(C2-Pad2): track 4.60 -> 0.00 mm
- net Net-(C47-Pad1): track 4.72 -> 0.76 mm
- net Net-(C36-Pad2): track 3.78 -> 0.00 mm
- net Net-(U2-BIAS): track 0.00 -> 3.74 mm
- net Net-(C28-Pad2): track 3.44 -> 0.00 mm
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Other:
- board text added: "0805 anti-pads"
- board text added: "2025-04-29"
- board text added: "SMA3109"
- board text added: "VCTRL"
- board text removed: "2025-04-11"
- board text removed: "BFP840"
- board text removed: "BGA8U1BN6"
- board text removed: "BGA9H1BN6"
- board text removed: "C1"
- board text removed: "C2"

Commit message: Update rf-amps board
Parts:
- removed C10, C12, C25, C55, C56, C60, C61, C62: 1 uF, Capacitor_SMD:C_0201_0603Metric
- removed C14, C16, C23, C24, C42: 220 nF, Capacitor_SMD:C_0201_0603Metric
- removed C47: C, Capacitor_SMD:C_0201_0603Metric
- removed L23: 47uH, Inductor_SMD:L_0603_1608Metric
- removed L24: 33nH, Inductor_SMD:L_0201_0603Metric
- removed L28, L29, L30, L31: 15 uH, Inductor_SMD:L_0603_1608Metric
- removed L32: L, Inductor_SMD:L_0805_2012Metric
- removed R2: 2.2k, Resistor_SMD:R_0201_0603Metric
- removed R36, R43: 360, Resistor_SMD:R_0201_0603Metric
- removed R37, R9: R, Resistor_SMD:R_0201_0603Metric
- removed R38, R39, R50, R51, R54, R55: 0, Resistor_SMD:R_0201_0603Metric
- removed U2, U3: BGB741L7ESD, rf-amps:TSLP-7-1
- removed U4: SMA3109, Package_TO_SOT_SMD:SOT-363_SC-70-6
- added C27: 1uF, Capacitor_SMD:C_0201_0603Metric, F.Cu at (144.8, 114.2)
- added C28: 1uF, Capacitor_SMD:C_0201_0603Metric, F.Cu at (144.8, 126.6)
- added C29: 1 uF, Capacitor_SMD:C_0201_0603Metric, F.Cu at (139.8, 115.7)
- added C30: 1 uF, Capacitor_SMD:C_0201_0603Metric, F.Cu at (139.6, 128.0)
- added C31: 1 uF, Capacitor_SMD:C_0201_0603Metric, F.Cu at (145.1, 116.6)
- added C32: 1 uF, Capacitor_SMD:C_0201_0603Metric, F.Cu at (144.8, 128.9)
- added C33: 1 uF, Capacitor_SMD:C_0201_0603Metric, F.Cu at (139.5, 139.3)
- added C34: 1uF, Capacitor_SMD:C_0201_0603Metric, F.Cu at (144.7, 138.2)
- added C35: 1 uF, Capacitor_SMD:C_0201_0603Metric, F.Cu at (144.1, 140.9)
- added C36: 1 uF, Capacitor_SMD:C_0201_0603Metric, F.Cu at (139.4, 151.3)
- added C37: 1uF, Capacitor_SMD:C_0201_0603Metric, F.Cu at (144.7, 150.2)
- added C38: 1 uF, Capacitor_SMD:C_0201_0603Metric, F.Cu at (144.7, 152.3)
- added C40: 0.3 pF, Capacitor_SMD:C_0201_0603Metric, F.Cu at (144.0, 80.0)
- added C52: 1 uF, Capacitor_SMD:C_0201_0603Metric, F.Cu at (141.3, 126.8)
- added C63: 1 uF, Capacitor_SMD:C_0201_0603Metric, F.Cu at (143.3, 81.4)
- added L12: 8.2 nH, Inductor_SMD:L_0201_0603Metric, F.Cu at (139.1, 79.7)
- added L25: 100 uH, Inductor_SMD:L_0805_2012Metric, F.Cu at (141.2, 81.5)
- added L26: 56 nH, Inductor_SMD:L_0201_0603Metric, F.Cu at (142.6, 80.0)
- added P9: CONN_01X03, Connector_PinHeader_2.54mm:PinHeader_1x03_P2.54mm_Vertical, F.Cu at (132.5, 146.0)
- added Q3: BFP840ESD, eval:SOT-343-4-3, F.Cu at (141.9, 116.3)
- added Q4: BFP840ESD, eval:SOT-343-4-3, F.Cu at (141.7, 128.7)
- added Q5: BFP840ESD, eval:SOT-343-4-3, F.Cu at (141.6, 140.0)
- added Q6: BFP840ESD, eval:SOT-343-4-3, F.Cu at (141.5, 152.0)
- added R11: 240, Resistor_SMD:R_0201_0603Metric, F.Cu at (142.6, 114.1)
- added R12: 75, Resistor_SMD:R_0201_0603Metric, F.Cu at (144.1, 126.6)
- added R13: 240, Resistor_SMD:R_0201_0603Metric, F.Cu at (142.3, 126.5)
- added R14: 75, Resistor_SMD:R_0201_0603Metric, F.Cu at (143.9, 138.2)
- added R15: 240, Resistor_SMD:R_0201_0603Metric, F.Cu at (142.9, 138.5)
- added R16: 27k, Resistor_SMD:R_0201_0603Metric, F.Cu at (140.2, 114.6)
- added R17: 27k, Resistor_SMD:R_0201_0603Metric, F.Cu at (139.9, 127.0)
- added R18: 51, Resistor_SMD:R_0201_0603Metric, F.Cu at (144.0, 116.2)
- added R20: 15, Resistor_SMD:R_0201_0603Metric, F.Cu at (144.0, 117.0)
- added R21: 51, Resistor_SMD:R_0201_0603Metric, F.Cu at (143.8, 128.6)
- added R22: 15, Resistor_SMD:R_0201_0603Metric, F.Cu at (143.8, 129.3)
- added R23: 27k, Resistor_SMD:R_0201_0603Metric, F.Cu at (139.8, 138.3)
- added R24: 51, Resistor_SMD:R_0201_0603Metric, F.Cu at (143.6, 139.6)
- added R25: 15, Resistor_SMD:R_0201_0603Metric, F.Cu at (143.3, 140.9)
- added R26: 27k, Resistor_SMD:R_0201_0603Metric, F.Cu at (141.2, 150.2)
- added R28: 75, Resistor_SMD:R_0201_0603Metric, F.Cu at (143.6, 149.9)
- added R30: 240, Resistor_SMD:R_0201_0603Metric, F.Cu at (143.2, 150.9)
- added R31: 15, Resistor_SMD:R_0201_0603Metric, F.Cu at (143.9, 152.3)
- added R40: 220, Resistor_SMD:R_0201_0603Metric, F.Cu at (142.9, 82.8)
- added R41: 220, Resistor_SMD:R_0201_0603Metric, F.Cu at (143.3, 80.0)
- C19, C20, C21, C22, C45, C46, C51: value 220 nF -> 1 uF
- C54: value C -> 1 uF
- L10, L14: value 1.8 nH -> 1.5 nH
- L11: value L -> 1.5 nH
- R10: value 470 -> 75
- R19: value 470 -> 180
- R27: value 2.2k -> 3.3k
- R29: value 2.2k -> 51
- R3, R6: value 4900 -> 33k
- R4, R7: value 330 -> 240
- R42: value 360 -> 300
- R44: value 0 -> 6.8k
- R49: value 0 -> 3
- R52, R53: value 3 -> 1
- moved R29 60.9 mm to (143.9, 150.9)
- moved C54 45.1 mm to (142.2, 150.5)
- moved C53 33.8 mm to (141.5, 138.5), turned to 180 degrees
- moved C17 24.0 mm to (143.6, 90.6), turned to 0 degrees
- moved C18 24.0 mm to (143.6, 102.6), turned to 0 degrees
- moved C19 24.0 mm to (143.9, 92.3)
- moved C20 24.0 mm to (139.4, 92.0)
- moved C21 24.0 mm to (139.4, 104.0)
- moved C22 24.0 mm to (143.9, 104.3)
- moved C45 24.0 mm to (140.4, 92.3)
- moved C46 24.0 mm to (140.4, 104.3)
- moved L10 24.0 mm to (142.6, 92.3)
- moved L14 24.0 mm to (142.6, 104.3)
- moved Q1 24.0 mm to (141.5, 91.7)
- moved Q2 24.0 mm to (141.5, 103.7)
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Connections:
- C17 pad 1: Net-(P6-Pin_2) -> Net-(P4-Pin_2)
- C18 pad 1: Net-(P7-Pin_2) -> Net-(P5-Pin_2)
- C19 pad 1: Net-(J8-In) -> Net-(J4-In)
- C20 pad 2: Net-(J7-In) -> Net-(J3-In)
- C21 pad 2: Net-(J9-In) -> Net-(J5-In)
- C22 pad 1: Net-(J10-In) -> Net-(J6-In)
- C51 pad 1: Net-(J4-In) -> Net-(C51-Pad1)
- R10 pad 1: Net-(U3-RFIN) -> Net-(P6-Pin_2)
- R19 pad 1: Net-(U1-RFIN) -> Net-(L12-Pad2)
- R29 pad 1: VCC -> Net-(R26-Pad1)
- R29 pad 2: Net-(U2-ADJ) -> Net-(L11-Pad2)
- R5 pad 2: Net-(P6-Pin_2) -> Net-(P4-Pin_2)
- R8 pad 2: Net-(P7-Pin_2) -> Net-(P5-Pin_2)
Routing:
- net Net-(P9-Pin_2): track 0.00 -> 11.2 mm
- net GND: track 14.0 -> 6.91 mm, vias 51 -> 84
- net Net-(R12-Pad2): track 0.00 -> 6.41 mm
- net Net-(R14-Pad2): track 0.00 -> 5.23 mm
- net Net-(R10-Pad2): track 1.53 -> 6.34 mm
- net VCC: track 8.63 -> 4.11 mm, vias 9 -> 3
- net Net-(Q4-C-Pad3): track 0.00 -> 4.40 mm
- net Net-(Q3-C-Pad3): track 0.00 -> 4.27 mm
- net Net-(U2-BIAS): track 3.74 -> 0.00 mm
- net Net-(Q5-C-Pad3): track 0.00 -> 3.21 mm
- net Net-(R26-Pad1): track 0.00 -> 3.17 mm
- net Net-(C63-Pad1): track 1.15 -> 4.05 mm
- net Net-(U2-RFOUT): track 2.77 -> 0.00 mm
- net Net-(U2-RFIN): track 2.71 -> 0.00 mm
- net Net-(Q4-B): track 0.00 -> 2.68 mm
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- added copper zone on F.Cu, net GND
Other:
- board text added: "2025-05-07"
- board text added: "BFP840"
- board text removed: "0805 anti-pads"
- board text removed: "2025-04-29"
- board text removed: "IN"
- board text removed: "OUT"
- board text removed: "SMA3109"

Commit message: Update rf-amps board
Parts:
- removed C11, C17, C18, C19, C20, C21, C22, C29, C30, C31, C32, C33, C35, C36, C38, C45, C46, C51, C52, C54, C57, C63: 1 uF, Capacitor_SMD:C_0201_0603Metric
- removed C15, C39: 220 nF, Capacitor_SMD:C_0201_0603Metric
- removed C27, C28, C34, C37: 1uF, Capacitor_SMD:C_0201_0603Metric
- removed C40: 0.3 pF, Capacitor_SMD:C_0201_0603Metric
- removed J10, J11, J12, J13, J14, J7, J8, J9: CONN_COAXIAL, sma-variants:SMA-EDGE-1.3mm-pad-1.05mm-gap-2.6mm-keepout
- removed L10, L11, L14: 1.5 nH, Inductor_SMD:L_0201_0603Metric
- removed P6, P7, P8, P9: CONN_01X03, Connector_PinHeader_2.54mm:PinHeader_1x03_P2.54mm_Vertical
- removed Q1: BFR840, eval:TSLP-3-9
- removed Q3, Q4, Q5, Q6: BFP840ESD, eval:SOT-343-4-3
- removed R10, R12, R14, R28: 75, Resistor_SMD:R_0201_0603Metric
- removed R11, R13, R15, R30, R4, R7: 240, Resistor_SMD:R_0201_0603Metric
- removed R16, R17, R23, R26: 27k, Resistor_SMD:R_0201_0603Metric
- removed R18, R21, R24, R29: 51, Resistor_SMD:R_0201_0603Metric
- removed R19: 180, Resistor_SMD:R_0201_0603Metric
- removed R20, R22, R25, R31: 15, Resistor_SMD:R_0201_0603Metric
- removed R27: 3.3k, Resistor_SMD:R_0201_0603Metric
- removed R3, R6: 33k, Resistor_SMD:R_0201_0603Metric
- removed R40, R41, R5, R8: 220, Resistor_SMD:R_0201_0603Metric
- removed R44: 6.8k, Resistor_SMD:R_0201_0603Metric
- removed R49: 3, Resistor_SMD:R_0201_0603Metric
- removed R52, R53: 1, Resistor_SMD:R_0201_0603Metric
- removed U1: BGB741L7ESD, rf-amps:TSLP-7-1
- added C114: 1 uF, Capacitor_SMD:C_0201_0603Metric, F.Cu at (139.5, 77.9)
- added C139: 1 uF, Capacitor_SMD:C_0201_0603Metric, F.Cu at (143.8, 81.4)
- added C160: 1 uF, Capacitor_SMD:C_0201_0603Metric, F.Cu at (140.7, 82.8)
- added C161: 1 uF, Capacitor_SMD:C_0201_0603Metric, F.Cu at (140.9, 78.0)
- added C185: 1 uF, Capacitor_SMD:C_0201_0603Metric, F.Cu at (142.1, 80.3)
- added C187: 0.3pF, Capacitor_SMD:C_0201_0603Metric, F.Cu at (145.9, 79.3)
- added C195: 1 uF, Capacitor_SMD:C_0201_0603Metric, F.Cu at (138.4, 123.7)
- added C196: 1 uF, Capacitor_SMD:C_0201_0603Metric, F.Cu at (142.2, 121.2)
- added C197: 1 uF, Capacitor_SMD:C_0201_0603Metric, F.Cu at (143.2, 122.9)
- added C198: 1 uF, Capacitor_SMD:C_0201_0603Metric, F.Cu at (143.9, 124.3)
- added C205: 1 uF, Capacitor_SMD:C_0201_0603Metric, F.Cu at (144.8, 121.5)
- added C206: 1 uF, Capacitor_SMD:C_0201_0603Metric, F.Cu at (143.3, 105.2)
- added C50: 1 uF, Capacitor_SMD:C_0201_0603Metric, F.Cu at (146.2, 102.0)
- added C62: 1 uF, Capacitor_SMD:C_0201_0603Metric, F.Cu at (145.2, 79.3)
- added C78: 1 uF, Capacitor_SMD:C_0201_0603Metric, F.Cu at (142.0, 102.7)
- added L28: 2.4 nH, Inductor_SMD:L_0201_0603Metric, F.Cu at (143.2, 124.3)
- added L5: 56 nH, Inductor_SMD:L_0201_0603Metric, F.Cu at (143.8, 102.3)
- added Q11: Q_PMOS_GSD, eval:TSLP-3-9, F.Cu at (144.1, 121.5)
- added Q14: Q_PMOS_GSD, eval:TSLP-3-9, F.Cu at (141.8, 105.1)
- added Q8: BFR840, eval:TSLP-3-9, F.Cu at (142.0, 101.7)
- added R114: 33k, Resistor_SMD:R_0201_0603Metric, F.Cu at (140.2, 102.3)
- added R115: 120, Resistor_SMD:R_0201_0603Metric, F.Cu at (143.1, 102.3)
- added R116: 120, Resistor_SMD:R_0201_0603Metric, F.Cu at (140.9, 102.3)
- added R117: 1, Resistor_SMD:R_0201_0603Metric, F.Cu at (144.8, 102.0)
- added R123: 12k, Resistor_SMD:R_0201_0603Metric, F.Cu at (141.2, 122.2)
- added R124: 180, Resistor_SMD:R_0201_0603Metric, F.Cu at (139.6, 79.0)
- added R126: 300, Resistor_SMD:R_0201_0603Metric, F.Cu at (140.7, 80.3)
- added R127: 3.3k, Resistor_SMD:R_0201_0603Metric, F.Cu at (142.3, 78.0)
- added R128: 6.8k, Resistor_SMD:R_0201_0603Metric, F.Cu at (142.1, 82.8)
- added R129: 220, Resistor_SMD:R_0201_0603Metric, F.Cu at (143.8, 80.0)
- added R131: 220, Resistor_SMD:R_0201_0603Metric, F.Cu at (143.4, 82.8)
- added R132: 1k, Resistor_SMD:R_0201_0603Metric, F.Cu at (142.2, 122.5)
- added R137: 100, Resistor_SMD:R_0201_0603Metric, F.Cu at (143.2, 121.5)
- added R138: 51, Resistor_SMD:R_0201_0603Metric, F.Cu at (143.9, 122.9)
- added R139: 10, Resistor_SMD:R_0201_0603Metric, F.Cu at (139.0, 123.7)
- added R140: 33k, Resistor_SMD:R_0201_0603Metric, F.Cu at (139.8, 123.7)
- added R141: 33k, Resistor_SMD:R_0201_0603Metric, F.Cu at (144.2, 119.8)
- added R146: 33k, Resistor_SMD:R_0201_0603Metric, F.Cu at (142.7, 105.2)
- added R43: 3, Resistor_SMD:R_0201_0603Metric, F.Cu at (144.2, 79.0)
- added U25: BGB741L7ESD, eval:TSLP-7-1, F.Cu at (141.5, 79.2)
- J1, J2, J3, J4, J5, J6: footprint sma-variants:SMA-EDGE-1.3mm-pad-1.05mm-gap-2.6mm-keepout -> eval:SMA_MyAntenna_A-SMA-KE-16.5A_EdgeMount
- L12: value 8.2 nH -> 56 nH
- L25: value 100 uH -> 8.2 nH; footprint Inductor_SMD:L_0805_2012Metric -> Inductor_SMD:L_0201_0603Metric
- L26: value 56 nH -> 100uH; footprint Inductor_SMD:L_0201_0603Metric -> eval:L_TDK_MLZ2012_h1.25mm
- Q2: value BFR840 -> BFP840; footprint eval:TSLP-3-9 -> eval:SOT-343-4-3
- R42: value 300 -> 220
- moved C53 34.8 mm to (140.2, 103.8), turned to 90 degrees
- moved R42 23.4 mm to (140.9, 103.8), turned to 90 degrees
- moved C58 21.8 mm to (139.2, 102.0)
- moved Q2 20.3 mm to (141.5, 124.0), turned to 0 degrees
- moved J5 20.0 mm to (130.0, 124.0)
- moved J6 20.0 mm to (153.0, 124.0)
- moved P5 15.0 mm to (132.5, 113.0)
- moved J3 10.0 mm to (130.0, 102.0)
- moved J4 10.0 mm to (153.0, 102.0)
- moved P4 5.00 mm to (132.5, 91.0)
- moved L12 4.07 mm to (143.1, 80.0), turned to 90 degrees
- moved C59 2.56 mm to (139.2, 80.3)
- moved L25 2.52 mm to (139.6, 79.7)
- moved L26 1.70 mm to (141.9, 81.5), turned to 0 degrees
Connections:
- C53 pad 1: Net-(C53-Pad1) -> Net-(Q14-S)
- C53 pad 2: Net-(Q5-B) -> GND
- C58 pad 1: Net-(C58-Pad1) -> Net-(J3-In)
- C58 pad 2: Net-(U1-RFOUT) -> Net-(Q8-B)
- C59 pad 1: GND -> Net-(J1-In)
- C59 pad 2: VCC -> Net-(U25-RFIN)
- L12 pad 1: Net-(U1-RFIN) -> Net-(C139-Pad1)
- L25 pad 1: Net-(C63-Pad1) -> Net-(U25-RFIN)
- L25 pad 2: VCC -> Net-(L25-Pad2)
- L26 pad 1: Net-(U1-RFOUT) -> VAA
- L26 pad 2: Net-(C63-Pad1) -> Net-(C139-Pad1)
- P2 pad 1: VCC -> VAA
- P2 pad 2: VCC -> VAA
- P3 pad 1: VCC -> VAA
- P4 pad 1: VCC -> VAA
- P5 pad 1: VCC -> VAA
- Q2 pad 2: Net-(Q2-C) -> GND
- Q2 pad 3: GND -> Net-(C198-Pad2)
- R42 pad 1: Net-(U1-RFIN) -> Net-(Q14-S)
- R42 pad 2: Net-(C58-Pad1) -> Net-(L5-Pad1)
Routing:
- net Net-(P7-Pin_2): track 11.5 -> 0.00 mm
- net Net-(P6-Pin_2): track 11.5 -> 0.00 mm
- net Net-(P9-Pin_2): track 11.2 -> 0.00 mm
- net Net-(P8-Pin_2): track 11.1 -> 0.00 mm
- net VAA: track 0.00 -> 8.11 mm, vias 0 -> 6
- net Net-(J7-In): track 7.47 -> 0.00 mm
- net Net-(J11-In): track 7.30 -> 0.00 mm
- net Net-(J13-In): track 7.20 -> 0.00 mm
- net Net-(J9-In): track 7.13 -> 0.00 mm
- net Net-(J12-In): track 7.06 -> 0.00 mm
- net Net-(J14-In): track 6.48 -> 0.00 mm
- net Net-(P4-Pin_2): track 10.9 -> 17.4 mm, vias 0 -> 1
- net Net-(R12-Pad2): track 6.41 -> 0.00 mm
- net Net-(R10-Pad2): track 6.34 -> 0.00 mm
- net Net-(J10-In): track 6.26 -> 0.00 mm
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- added copper zone on In2.Cu, net VAA
- removed copper zone on In2.Cu, net VCC
Other:
- board size 23 x 100 mm -> 23 x 75 mm
- board text added: "2025-06-16"
- board text added: "VAA"
- board text removed: "2025-05-07"
- board text removed: "VCC"
