File: evaluation-boards/rf-amps/rf-amps.kicad_sch (KiCad schematic)
At the start: 16 parts, among them J1 Conn_01x02, J2 Conn_01x02, J3 CONN_01X03, J4 CONN_COAXIAL, J5 CONN_COAXIAL, U1 BGB741L7ESD

Commit message: Add more amplifiers to rf-amps board
Parts:
- added C10, C11, C12, C13, C14, C15, C16, C17, C18, C19, C20, C22, C23, C24, C30, C34, C35, C37, C38, C39, C40, C41, C42, C43, C44, C5, C6, C7, C8: 1uF, Capacitor_SMD:C_0201_0603Metric, symbol Device:C
- added C21, C31: 0.2pF, Capacitor_SMD:C_0201_0603Metric, symbol Device:C
- added C25, C27, C28, C29, C33, C36: C, Capacitor_SMD:C_0201_0603Metric, symbol Device:C
- added C26, C32: 100pF, Capacitor_SMD:C_0201_0603Metric, symbol Device:C
- added J10, J11, J12, J13, J15, J16, J17, J19, J21, J6, J7, J9: CONN_COAXIAL, sma-variants:Linx_SMA_CONSMA003.062, symbol Connector:Conn_Coaxial
- added J14, J18, J20, J22, J23, J24, J25, J8: CONN_01X03, Connector_PinHeader_2.54mm:PinHeader_1x03_P2.54mm_Vertical, symbol Connector_Generic:Conn_01x03
- added L10, L13, L15, L5, L8: 33nH, Inductor_SMD:L_0201_0603Metric, symbol Device:L
- added L11, L14, L16, L6, L9: 47uH, Inductor_SMD:L_0603_1608Metric, symbol Device:L
- added L12, L7: L, Inductor_SMD:L_0201_0603Metric, symbol Device:L
- added R2: 0, Resistor_SMD:R_0402_1005Metric, symbol Device:R
- added R3: 24, Resistor_SMD:R_0402_1005Metric, symbol Device:R
- added R4: 10k, Resistor_SMD:R_0402_1005Metric, symbol Device:R
- added R5: 33k, Resistor_SMD:R_0402_1005Metric, symbol Device:R
- added R6, R7: R, Resistor_SMD:R_0201_0603Metric, symbol Device:R
- added R8, R9: 900, Resistor_SMD:R_0402_1005Metric, symbol Device:R
- added U10, U7: SKY13453, gsg-modules:SKY13350-385LF, symbol gsg-symbols:SKY13453
- added U2: TRF37A73, Package_SON:WSON-8-1EP_2x2mm_P0.5mm_EP0.9x1.6mm, symbol rf-amps:TRF37A73
- added U3: BGA2817, Package_TO_SOT_SMD:SOT-363_SC-70-6, symbol RF_Amplifier:BGA2817
- added U4: TQP369184, Package_TO_SOT_SMD:SOT-363_SC-70-6, symbol rf-amps:TQP369184
- added U5: TQP3M9037, Package_SON:WSON-8-1EP_2x2mm_P0.5mm_EP0.9x1.6mm, symbol rf-amps:TQP3M9037
- added U6, U8: GRF4001, rf-amps:DFN-6-1EP_1.5x1.5mm_P0.5mm_EP0.6x1.1mm, symbol rf-amps:GRF4001
Connections:
- net GND: now also C10.1, C11.1, C15.1, C17.1, C18.1, C21.1, C24.1, C25.2, C26.1, C27.2, C28.2, C29.2, C31.1, C32.1, C33.2, C34.1, C36.2, C41.1, C42.1, C43.1, C44.1, C6.1, C8.1, J10.2 (Ext), J11.2 (Ext), J12.2 (Ext), J13.2 (Ext), J14.3 (Pin_3), J15.2 (Ext), J16.2 (Ext), J17.2 (Ext), J18.3 (Pin_3), J19.2 (Ext), J20.3 (Pin_3), J21.2 (Ext), J22.3 (Pin_3), J23.3 (Pin_3), J24.3 (Pin_3), J25.3 (Pin_3), J6.2 (Ext), J7.2 (Ext), J8.3 (Pin_3), J9.2 (Ext), L12.1, R4.1, R6.2, U10.3 (GND), U2.3 (NC), U2.4 (NC), U2.6 (NC), U2.8 (NC), U2.9 (GND), U3.2 (G), U3.4 (G), U3.5 (G), U4.1 (GND), U4.2 (GND), U4.4 (GND), U4.5 (GND), U5.1 (NC), U5.3 (NC), U5.4 (NC), U5.5 (NC), U5.8 (NC), U5.9 (GND), U6.2 (NC), U6.5 (NC), U6.6 (NC), U6.7 (GND), U7.3 (GND), U8.2 (NC), U8.5 (NC), U8.6 (NC), U8.7 (GND)
- net VCC: now also C10.2, C18.2, C24.2, C34.2, C41.2, C42.2, C8.2, J14.1 (Pin_1), J18.1 (Pin_1), J20.1 (Pin_1), J22.1 (Pin_1), J23.1 (Pin_1), J24.1 (Pin_1), J25.1 (Pin_1), J8.1 (Pin_1), L11.2, L14.2, L16.2, R2.2, R7.1, U10.1 (VDD), U2.1 (VCC), U7.1 (VDD)
- new net: C16.1, J12.1 (In)
- new net: C16.2, L8.1, U4.6
- new net: J14.2 (Pin_2), R5.1
- new net: R4.2, R5.2, U5.6 (SHUTDOWN)
- new net: C19.2, L10.1, U5.7 (RFOUT)
- new net: L10.2, L11.1
- new net: C11.2, J24.2 (Pin_2), L7.1, L7.2, U3.1 (Vcc)
- new net: C20.2, J13.1 (In), L12.2
- new net: J18.2 (Pin_2), R8.1
- new net: C26.2, R8.2, U6.1 (VEN)
- new net: C19.1, J15.1 (In)
- new net: C7.1, J7.1 (In)
- new net: C37.1, U10.6 (RFC)
- new net: C37.2, J19.1 (In)
- new net: C5.1, U2.2 (RFIN)
- new net: J8.2 (Pin_2), U2.5 (PWDN)
- new net: C7.2, L5.1, U2.7 (RFOUT)
- new net: C21.2, C22.1, U6.3 (RFIN)
- new net: C23.2, C25.1, L13.1, U6.4 (RFOUT)
- new net: C14.1, U4.3
- new net: C13.1, J10.1 (In)
- new net: C13.2, U3.3
- new net: C35.1, C36.1, C40.1, U10.4 (RF2)
- new net: C6.2, L6.2, R2.1
- new net: C5.2, J6.1 (In)
- new net: C43.2, J22.2 (Pin_2), U10.5 (VCTL)
- new net: C44.2, J23.2 (Pin_2), U7.5 (VCTL)
- new net: C17.2, J25.2 (Pin_2), R3.2
- new net: C14.2, J11.1 (In)
- new net: C30.1, C31.2, U8.3 (RFIN)
- new net: C12.2, J9.1 (In)
- new net: C23.1, C27.1, J17.1 (In)
- new net: C20.1, R6.1, R7.2, U5.2 (RFIN)
- new net: C15.2, L9.2, R3.1
- new net: C38.1, J21.1 (In)
- new net: L13.2, L14.1
- new net: C29.1, C30.2, C39.1, U10.2 (RF1)
- new net: C22.2, C28.1, J16.1 (In)
- new net: L15.2, L16.1
- new net: C33.1, C35.2, L15.1, U8.4 (RFOUT)
- new net: C39.2, U7.4 (RF2)
- new net: L8.2, L9.1
- new net: L5.2, L6.1
- new net: C40.2, U7.2 (RF1)
- new net: C38.2, U7.6 (RFC)
- new net: C12.1, U3.6
- new net: J20.2 (Pin_2), R9.1
- new net: C32.2, R9.2, U8.1 (VEN)
Other:
- note added: "24 ohms recommended for 5 V supply. Higher resistance for higher voltage."
- note added: "R2 3.9 ohms for TRF37B73"
- moved on the sheet: C1, C2, C3, C4, C9, J1, J2, J3, J4, J5, L1, L2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

Commit message: Update TSLP-7-1 footprint
Parts:
- U1: footprint gsg-modules:TSLP-7-1 -> rf-amps:TSLP-7-1
Changed lines of the file:
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@@
 			)
 		)
-		(property "Footprint" "gsg-modules:TSLP-7-1"
+		(property "Footprint" "rf-amps:TSLP-7-1"
 			(at 83.82 64.77 0)
 			(effects

Commit message: Update rf-amps board
Parts:
- removed C11, C12, C13, C15, C3, C39, C42: 1uF, Capacitor_SMD:C_0201_0603Metric, symbol Device:C
- removed J20, J23, J8: CONN_01X03, Connector_PinHeader_2.54mm:PinHeader_1x03_P2.54mm_Vertical, symbol Connector_Generic:Conn_01x03
- removed L1, L14, L16, L2, L6, L9: 47uH, Inductor_SMD:L_0603_1608Metric, symbol Device:L
- removed L15, L4, L5: 33nH, Inductor_SMD:L_0201_0603Metric, symbol Device:L
- removed L7: L, Inductor_SMD:L_0201_0603Metric, symbol Device:L
- removed U1: BGB741L7ESD, rf-amps:TSLP-7-1, symbol gsg-symbols:BGB741L7ESD
- removed U10, U7: SKY13453, gsg-modules:SKY13350-385LF, symbol gsg-symbols:SKY13453
- removed U2: TRF37A73, Package_SON:WSON-8-1EP_2x2mm_P0.5mm_EP0.9x1.6mm, symbol rf-amps:TRF37A73
- removed U3: BGA2817, Package_TO_SOT_SMD:SOT-363_SC-70-6, symbol RF_Amplifier:BGA2817
- removed U4: TQP369184, Package_TO_SOT_SMD:SOT-363_SC-70-6, symbol rf-amps:TQP369184
- removed U5: TQP3M9037, Package_SON:WSON-8-1EP_2x2mm_P0.5mm_EP0.9x1.6mm, symbol rf-amps:TQP3M9037
- removed U6, U8: GRF4001, rf-amps:DFN-6-1EP_1.5x1.5mm_P0.5mm_EP0.6x1.1mm, symbol rf-amps:GRF4001
- added C45, C46, C47, C48: 39pF, Capacitor_SMD:C_0201_0603Metric, symbol Device:C
- added C49, C50, C53, C54, C56: C, Capacitor_SMD:C_0201_0603Metric, symbol Device:C
- added C55: 1uF, Capacitor_SMD:C_0201_0603Metric, symbol Device:C
- added L17, L19, L23: 47uH, Inductor_SMD:L_0603_1608Metric, symbol Device:L
- added L18, L20, L24: 33nH, Inductor_SMD:L_0201_0603Metric, symbol Device:L
- added L25, L26, L27: L, Inductor_SMD:L_0201_0603Metric, symbol Device:L
- added P4: CONN_02X03, Connector_PinHeader_2.54mm:PinHeader_2x03_P2.54mm_Vertical, symbol Connector_Generic:Conn_02x03_Odd_Even
- added Q1, Q2: BFR840, eval:TSLP-3-9, symbol Transistor_BJT:Q_NPN_BCE
- added Q3, Q4: BFP840ESD, eval:SOT-343-4-3, symbol eval:Q_NPN_BECE
- added R11, R25, R36, R37: R, Resistor_SMD:R_0201_0603Metric, symbol Device:R
- added R12: 33k, Resistor_SMD:R_0201_0603Metric, symbol Device:R
- added R13: 27, Resistor_SMD:R_0201_0603Metric, symbol Device:R
- added R14, R15, R19, R24, R26, R38, R39, R40, R45, R46, R47, R48: 0, Resistor_SMD:R_0201_0603Metric, symbol Device:R
- added R16, R21: 30k, Resistor_SMD:R_0201_0603Metric, symbol Device:R
- added R17, R18, R22: 82, Resistor_SMD:R_0201_0603Metric, symbol Device:R
- added R20, R23: 10, Resistor_SMD:R_0201_0603Metric, symbol Device:R
- added U1: BGA9H1BN6, eval:TSLP-6-4_1.1x0.7mm_P0.4mm, symbol rf-amps:BGA9H1BN6
- added U2: BGA8U1BN6, eval:TSLP-6-4_1.1x0.7mm_P0.4mm, symbol rf-amps:BGA8U1BN6
- added U4: BGB741L7ESD, rf-amps:TSLP-7-1, symbol gsg-symbols:BGB741L7ESD
- C18, C23: value 1uF -> 1pF
- C19, C24: value 1uF -> 18pF
- C20, C22: value 1uF -> 22pF
- C21: value 0.2pF -> 1uF
- C26: value 100pF -> C
- C27, C33: value C -> 1uF; now fitted
- C28: value C -> 39pF; now fitted
- C29: value C -> 3.3pF; now fitted
- C30: value 1uF -> 1pF; now not fitted
- C31: value 0.2pF -> 10pF
- C32: value 100pF -> 10pF; now fitted
- C34: value 1uF -> 39pF
- C35: value 1uF -> 3.3pF
- C36: value C -> 1pF
- C37, C38: value 1uF -> 10pF
- C4, C40, C41, C43, C44, C6: value 1uF -> C; now not fitted
- L10: value 33nH -> 3.7nH
- L11: value 47uH -> 2.2nH; footprint Inductor_SMD:L_0603_1608Metric -> Inductor_SMD:L_0201_0603Metric
- L12: value L -> 5.1nH; now fitted
- L13: value 33nH -> 5.1nH
- L3: value 33nH -> 4.7 nH
- L8: value 33nH -> L
- P3: renamed from J3; value CONN_01X03 -> CONN_02X03; footprint Connector_PinHeader_2.54mm:PinHeader_1x03_P2.54mm_Vertical -> Connector_PinHeader_2.54mm:PinHeader_2x03_P2.54mm_Vertical; symbol Connector_Generic:Conn_01x03 -> Connector_Generic:Conn_02x03_Odd_Even
- R1: value 3k -> 0; footprint Resistor_SMD:R_0402_1005Metric -> Resistor_SMD:R_0201_0603Metric; now not fitted
- R2: value 0 -> R; footprint Resistor_SMD:R_0402_1005Metric -> Resistor_SMD:R_0201_0603Metric
- R3: value 24 -> 33k; footprint Resistor_SMD:R_0402_1005Metric -> Resistor_SMD:R_0201_0603Metric
- R4: value 10k -> 120; footprint Resistor_SMD:R_0402_1005Metric -> Resistor_SMD:R_0201_0603Metric
- R5: value 33k -> 27; footprint Resistor_SMD:R_0402_1005Metric -> Resistor_SMD:R_0201_0603Metric
- R6: value R -> 0; now fitted
- R7: value R -> 120; now fitted
- R8: value 900 -> 0; footprint Resistor_SMD:R_0402_1005Metric -> Resistor_SMD:R_0201_0603Metric
- R9: value 900 -> 82; footprint Resistor_SMD:R_0402_1005Metric -> Resistor_SMD:R_0201_0603Metric
- renumbered J4 to J1, J15 to J10, J16 to J11, J17 to J12, J19 to J13, J21 to J14, J5 to J2, J6 to J3, J7 to J4, J9 to J5, J10 to J6, J11 to J7, J12 to J8, J13 to J9, J2 to P1, J1 to P2, J24 to P5, J25 to P6, J14 to P7, J18 to P8, J22 to P9
Connections:
- net GND: now also C17.2, C21.2, C23.1, C25.1, C28.1, C30.1, C32.2, C36.1, C38.2, C40.2, C41.2, C43.2, C44.2, P3.5 (Pin_5), P3.6 (Pin_6), R1.2, C45.2, C46.2, C47.2, C48.2, C49.2, C50.2, C55.1, C56.2, L25.2, L26.2, L27.2, P4.5 (Pin_5), P4.6 (Pin_6), Q1.3 (E), Q3.2 (E), Q3.4 (C), R11.2, R14.2, R24.2, R25.2, R37.2, R40.2, U1.1 (GND), U2.5 (GND), U4.7 (GND); no longer C17.1, C21.1, C24.1, C25.2, C28.2, C29.2, C31.1, C32.1, C36.2, C4.1, C41.1, C43.1, C44.1, C6.1, L12.1, P3.3 (Pin_3), R4.1, R6.2
- net VCC: now also P3.2 (Pin_2), R2.1, C55.2, P4.1 (Pin_1), P4.2 (Pin_2), R38.2, U1.2 (VCC), U2.2 (VCC), U4.1 (VCC); no longer C18.2, C24.2, C34.2, C4.2, C41.2, L11.2, R1.1, R2.2, R7.1
- net at C2.2: now also U1.3
- net at L3.2: now also U1.5
- net at C16.1: now also J6.1 (In); no longer J8.1 (In)
- net at C16.2: now also R39.1; no longer L8.1
- net at R5.1: now also R4.2, R6.1, C45.1; no longer P7.2 (Pin_2)
- net at R5.2: now also C18.2, L10.1; no longer R4.2
- net at C19.2: now also L10.2, Q1.2 (C); no longer L10.1
- net at L11.1: now also C30.2, R18.2; no longer L10.2
- net at P5.2 (Pin_2): now also U4.5 (VCTRL)
- net at P8.2 (Pin_2): now also C27.1, R9.1; no longer R8.1
- net at C26.2, R8.2: now also R12.1
- net at C19.1: now also J8.1 (In); no longer J10.1 (In)
- net at C37.1: now also C38.1, J14.1 (In)
- net at C37.2: now also R46.2; no longer J13.1 (In)
- net at C5.1: now also U2.6
- net at C7.2: now also U2.3
- net at C22.1: now also C43.1, Q2.1 (B), R12.2; no longer C21.2
- net at C14.1: now also L8.1, R36.1, U4.3 (RFIN)
- net at C6.2: now also R25.1; no longer R2.1
- net at P9.2 (Pin_2): now also C33.1, C50.1, R17.1, R26.2; no longer C43.2
- net at C14.2: now also J5.1 (In); no longer J7.1 (In)
- net at C31.2: now also R45.2; no longer C30.1
- net at R3.1: now also C25.2, R6.2
- net at L13.2: now also C35.1, C41.1, Q4.1 (B)
- net at C29.1: now also C40.1, L12.2, Q3.1 (B); no longer C30.2
- net at C35.2: now also J13.1 (In), L26.1; no longer C33.1
- net at L8.2: now also C56.1, U4.2 (BIAS)
- net at R9.2: now also C47.1, R16.1, R18.1; no longer C32.2
- new net: P3.3 (Pin_3), R19.1
- new net: P3.4 (Pin_4), U1.6 (C1)
- new net: Q4.2 (E), R24.1
- new net: L20.1, Q4.3 (C), R23.1
- new net: Q4.4 (C), R40.1
- new net: C6.1, L19.1, L20.2
- new net: C4.2, R11.1
- new net: C48.1, R17.2, R21.1, R22.1
- new net: C34.2, L13.1, R21.2
- new net: P4.3 (Pin_3), U2.1 (C2)
- new net: P4.4 (Pin_4), U2.4 (C1)
- new net: C4.1, L17.1, L18.2
- new net: C22.2, J9.1 (In), L27.1
- new net: L18.1, Q2.2 (C), R48.1
- new net: Q2.3 (E), R14.1
- new net: C36.2, L19.2, R22.2, R26.1
- new net: R23.2, R46.1
- new net: C53.2, L24.1, R39.2, U4.4 (RFOUT)
- new net: C54.1, L23.1, L24.2
- new net: L11.2, Q3.3 (C), R20.1
- new net: R2.2, U4.6 (ADJ)
- new net: C53.1, R36.2
- new net: R47.1, R48.2
- new net: C24.2, R47.2
- new net: C23.2, L17.2, R13.2, R15.1
- new net: C21.1, C49.1, P7.2 (Pin_2), R15.2, R7.1
- new net: C29.2, J11.1 (In), L25.1
- new net: C17.1, P6.2 (Pin_2), R4.1
- new net: C20.2, J7.1 (In)
- new net: C28.2, L12.1, R16.2
- new net: C24.1, C44.1, J10.1 (In)
- new net: C20.1, Q1.1 (B), R3.2
- new net: C46.1, R13.1, R7.2, R8.1
- new net: L23.2, R38.1
- new net: C31.1, C32.1, J12.1 (In)
- new net: C54.2, R37.1
- new net: R20.2, R45.1
- new net: R1.1, R19.2, U1.4 (C2)
Other:
- note added: "install R1 instead of R19 for BGA5H1BN6 or BGA7H1BN6"
- note removed: "24 ohms recommended for 5 V supply. Higher resistance for higher voltage."
- note removed: "R2 3.9 ohms for TRF37B73"
- moved on the sheet: C1, C14, C16, C18, C19, C2, C20, C25, C5, C7, C8, C9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

Commit message: Update rf-amps board
Parts:
- removed C1, C2, C27, C33, C5, C7, C8, C9: 1uF, Capacitor_SMD:C_0201_0603Metric, symbol Device:C
- removed C26, C4, C40, C41, C43, C44, C49, C50, C6: C, Capacitor_SMD:C_0201_0603Metric, symbol Device:C
- removed C28, C34, C48: 39pF, Capacitor_SMD:C_0201_0603Metric, symbol Device:C
- removed C29, C35: 3.3pF, Capacitor_SMD:C_0201_0603Metric, symbol Device:C
- removed C30, C36: 1pF, Capacitor_SMD:C_0201_0603Metric, symbol Device:C
- removed C31, C32, C37, C38: 10pF, Capacitor_SMD:C_0201_0603Metric, symbol Device:C
- removed L12, L13: 5.1nH, Inductor_SMD:L_0201_0603Metric, symbol Device:L
- removed L17, L19: 47uH, Inductor_SMD:L_0603_1608Metric, symbol Device:L
- removed L18, L20: 33nH, Inductor_SMD:L_0201_0603Metric, symbol Device:L
- removed L25, L26, L27, L8: L, Inductor_SMD:L_0201_0603Metric, symbol Device:L
- removed L3: 4.7 nH, Inductor_SMD:L_0201_0603Metric, symbol Device:L
- removed P3, P4: CONN_02X03, Connector_PinHeader_2.54mm:PinHeader_2x03_P2.54mm_Vertical, symbol Connector_Generic:Conn_02x03_Odd_Even
- removed P9: CONN_01X03, Connector_PinHeader_2.54mm:PinHeader_1x03_P2.54mm_Vertical, symbol Connector_Generic:Conn_01x03
- removed Q3, Q4: BFP840ESD, eval:SOT-343-4-3, symbol eval:Q_NPN_BECE
- removed R1, R14, R15, R24, R26, R40, R45, R46, R47, R48: 0, Resistor_SMD:R_0201_0603Metric, symbol Device:R
- removed R11, R25: R, Resistor_SMD:R_0201_0603Metric, symbol Device:R
- removed R12: 33k, Resistor_SMD:R_0201_0603Metric, symbol Device:R
- removed R13: 27, Resistor_SMD:R_0201_0603Metric, symbol Device:R
- removed R16, R21: 30k, Resistor_SMD:R_0201_0603Metric, symbol Device:R
- removed R17, R18, R22: 82, Resistor_SMD:R_0201_0603Metric, symbol Device:R
- removed R20, R23: 10, Resistor_SMD:R_0201_0603Metric, symbol Device:R
- removed U1: BGA9H1BN6, eval:TSLP-6-4_1.1x0.7mm_P0.4mm, symbol rf-amps:BGA9H1BN6
- removed U2: BGA8U1BN6, eval:TSLP-6-4_1.1x0.7mm_P0.4mm, symbol rf-amps:BGA8U1BN6
- added C11, C12, C57, C58, C59, C60, C61, C62: 1 uF, Capacitor_SMD:C_0201_0603Metric, symbol Device:C
- added C15, C39, C42, C51: 220 nF, Capacitor_SMD:C_0201_0603Metric, symbol Device:C
- added L14: 1.8 nH, Inductor_SMD:L_0201_0603Metric, symbol Device:L
- added L28, L29, L30, L31: 15 uH, Inductor_SMD:L_0603_1608Metric, symbol Device:L
- added L32: L, Inductor_SMD:L_0805_2012Metric, symbol Device:L
- added P3, P4: CONN_01X03, Connector_PinHeader_2.54mm:PinHeader_1x03_P2.54mm_Vertical, symbol Connector_Generic:Conn_01x03
- added R10: 470, Resistor_SMD:R_0201_0603Metric, symbol Device:R
- added R27, R29: 2.2k, Resistor_SMD:R_0201_0603Metric, symbol Device:R
- added R42, R43: 360, Resistor_SMD:R_0201_0603Metric, symbol Device:R
- added R44, R49, R50, R51, R54, R55: 0, Resistor_SMD:R_0201_0603Metric, symbol Device:R
- added R52, R53: 3, Resistor_SMD:R_0201_0603Metric, symbol Device:R
- added U1, U2: BGB741L7ESD, rf-amps:TSLP-7-1, symbol gsg-symbols:BGB741L7ESD
- added U4: SMA3109, Package_TO_SOT_SMD:SOT-363_SC-70-6, symbol RF_Amplifier:BGA2866
- C10, C17: value 1uF -> 1 uF
- C14, C16, C21: value 1uF -> 220 nF
- C18: value 1pF -> 1 uF
- C19, C24: value 18pF -> 220 nF
- C20, C22: value 22pF -> 220 nF
- C23: value 1pF -> 220 nF
- C25, C53, C56: value C -> 1 uF; now fitted
- C45, C46: value 39pF -> 220 nF
- C47: value 39pF -> C; now not fitted
- C55: value 1uF -> 1 uF; now fitted
- J1, J10, J11, J12, J13, J14, J2, J3, J4, J5, J6, J7, J8, J9: footprint sma-variants:Linx_SMA_CONSMA003.062 -> sma-variants:SMA-EDGE-1.3mm-pad-1.05mm-gap-2.6mm-keepout
- L10: value 3.7nH -> 1.8 nH
- L11: value 2.2nH -> L; now not fitted
- L23, L24, R38: now fitted
- R19: value 0 -> 470
- R2: value R -> 2.2k
- R3: value 33k -> 4900
- R36: value R -> 360; now fitted
- R4, R7: value 120 -> 330
- R5: value 27 -> 220
- R6: value 0 -> 4900
- R8: value 0 -> 220
- R9: value 82 -> R; now not fitted
- renumbered U4 to U3
Connections:
- net GND: now also C18.2, C25.2, Q2.3 (E), C11.1, C12.1, C57.2, C59.1, C60.2, C62.1, P3.3 (Pin_3), P4.3 (Pin_3), U1.7 (GND), U2.7 (GND), U4.2 (G), U4.4 (G), U4.5 (G); no longer C18.1, C21.2, C23.1, C25.1, C45.2, C46.2, C47.2
- net VCC: now also C11.2, C12.2, C59.2, C62.2, P3.1 (Pin_1), P4.1 (Pin_1), R27.1, R29.1, R44.2, R50.2, U1.1 (VCC), U2.1 (VCC)
- net at J2.1 (In): now also C39.1
- net at J1.1 (In): now also C15.2
- net at R19.1: now also C15.1, R42.1, U1.3 (RFIN)
- net at R8.2: now also C18.1, P7.2 (Pin_2)
- net at Q2.1 (B): now also C21.1, C46.2, R6.1; no longer C22.1
- net at L10.2, Q1.2 (C): now also R3.2, R5.1, R52.2; no longer C19.2
- net at J9.1 (In): now also C21.2; no longer C22.2
- net at Q2.2 (C): now also R6.2, R8.1, L14.2, R53.2
- net at C47.1: now also R9.1; no longer R9.2
- net at L11.1: now also R9.2
- net at J4.1 (In): now also C51.1
- net at L11.2: now also L31.1, R55.1, U4.3
- net at C14.1, R36.1, U3.3 (RFIN): now also R10.1
- net at C24.2: now also R55.2
- net at J13.1 (In): now also L32.2
- net at C23.2: now also J11.1 (In)
- net at J14.1 (In): now also L32.1
- net at J3.1 (In): now also C42.2
- net at C17.1, P6.2 (Pin_2): now also R5.2; no longer R4.1
- net at P8.2 (Pin_2): now also C25.1, R54.1, U4.1 (Vcc); no longer R9.1
- net at J10.1 (In): now also C22.1; no longer C24.1
- net at C20.1, Q1.1 (B): now also C45.2, R3.1; no longer R3.2
- net at C56.1, U3.2 (BIAS): now also R10.2
- net at J12.1 (In): now also C24.1
- net at R19.2: now also C57.1, U1.2 (BIAS)
- new net: C23.1, C47.2, U4.6
- new net: L10.1, R4.2
- new net: C19.2, R52.1
- new net: C60.1, L30.2, U2.2 (BIAS)
- new net: C42.1, L30.1, R43.1, U2.3 (RFIN)
- new net: C61.2, L29.1, R51.2, U2.4 (RFOUT)
- new net: P4.2 (Pin_2), U2.5 (VCTRL)
- new net: R29.2, U2.6 (ADJ)
- new net: C51.2, R51.1
- new net: L14.1, R7.2
- new net: C61.1, R43.2
- new net: C58.1, R42.2
- new net: C46.1, R7.1
- new net: C22.2, R53.1
- new net: C39.2, R49.1
- new net: C58.2, L28.1, R49.2, U1.4 (RFOUT)
- new net: L28.2, R44.1
- new net: L31.2, R54.2
- new net: P3.2 (Pin_2), U1.5 (VCTRL)
- new net: R27.2, U1.6 (ADJ)
- new net: C45.1, R4.1
- new net: L29.2, R50.1
Other:
- note removed: "install R1 instead of R19 for BGA5H1BN6 or BGA7H1BN6"
- moved on the sheet: C16, C17, C19, C20, C45, C54, J1, J10, J12, J13, J14, J2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

Commit message: Update rf-amps board
Parts:
- removed C10, C12, C25, C55, C56, C60, C61, C62: 1 uF, Capacitor_SMD:C_0201_0603Metric, symbol Device:C
- removed C14, C16, C23, C24, C42: 220 nF, Capacitor_SMD:C_0201_0603Metric, symbol Device:C
- removed C47: C, Capacitor_SMD:C_0201_0603Metric, symbol Device:C
- removed L23: 47uH, Inductor_SMD:L_0603_1608Metric, symbol Device:L
- removed L24: 33nH, Inductor_SMD:L_0201_0603Metric, symbol Device:L
- removed L28, L29, L30, L31: 15 uH, Inductor_SMD:L_0603_1608Metric, symbol Device:L
- removed L32: L, Inductor_SMD:L_0805_2012Metric, symbol Device:L
- removed R2: 2.2k, Resistor_SMD:R_0201_0603Metric, symbol Device:R
- removed R36, R43: 360, Resistor_SMD:R_0201_0603Metric, symbol Device:R
- removed R37, R9: R, Resistor_SMD:R_0201_0603Metric, symbol Device:R
- removed R38, R39, R50, R51, R54, R55: 0, Resistor_SMD:R_0201_0603Metric, symbol Device:R
- removed U2, U3: BGB741L7ESD, rf-amps:TSLP-7-1, symbol gsg-symbols:BGB741L7ESD
- removed U4: SMA3109, Package_TO_SOT_SMD:SOT-363_SC-70-6, symbol RF_Amplifier:BGA2866
- added C27, C28, C34, C37: 1uF, Capacitor_SMD:C_0201_0603Metric, symbol Device:C
- added C29, C30, C31, C32, C33, C35, C36, C38, C52, C63: 1 uF, Capacitor_SMD:C_0201_0603Metric, symbol Device:C
- added C40: 0.3 pF, Capacitor_SMD:C_0201_0603Metric, symbol Device:C
- added L12: 8.2 nH, Inductor_SMD:L_0201_0603Metric, symbol Device:L
- added L25: 100 uH, Inductor_SMD:L_0805_2012Metric, symbol Device:L
- added L26: 56 nH, Inductor_SMD:L_0201_0603Metric, symbol Device:L
- added P9: CONN_01X03, Connector_PinHeader_2.54mm:PinHeader_1x03_P2.54mm_Vertical, symbol Connector_Generic:Conn_01x03
- added Q3, Q4, Q5, Q6: BFP840ESD, eval:SOT-343-4-3, symbol eval:Q_NPN_BECE
- added R11, R13, R15, R30: 240, Resistor_SMD:R_0201_0603Metric, symbol Device:R
- added R12, R14, R28: 75, Resistor_SMD:R_0201_0603Metric, symbol Device:R
- added R16, R17, R23, R26: 27k, Resistor_SMD:R_0201_0603Metric, symbol Device:R
- added R18, R21, R24: 51, Resistor_SMD:R_0201_0603Metric, symbol Device:R
- added R20, R22, R25, R31: 15, Resistor_SMD:R_0201_0603Metric, symbol Device:R
- added R40, R41: 220, Resistor_SMD:R_0201_0603Metric, symbol Device:R
- C19, C20, C21, C22, C45, C46, C51: value 220 nF -> 1 uF
- C54: value C -> 1 uF; now fitted
- L10, L14: value 1.8 nH -> 1.5 nH
- L11: value L -> 1.5 nH; now fitted
- R10: value 470 -> 75
- R19: value 470 -> 180
- R27: value 2.2k -> 3.3k
- R29: value 2.2k -> 51
- R3, R6: value 4900 -> 33k
- R4, R7: value 330 -> 240
- R42: value 360 -> 300
- R44: value 0 -> 6.8k
- R49: value 0 -> 3
- R52, R53: value 3 -> 1
Connections:
- net GND: now also C27.2, C28.2, C34.2, C37.2, C40.2, P9.3 (Pin_3), Q3.2 (E), Q3.4 (C), Q4.2 (E), Q4.4 (C), Q5.2 (E), Q5.4 (C), Q6.2 (E), Q6.4 (C), R40.2
- net VCC: now also L25.2, P9.1 (Pin_1); no longer R29.1
- net at C39.1, J2.1 (In): now also C40.1
- net at J6.1 (In): now also C22.1
- net at J11.1 (In): now also C33.2
- net at C17.1, R5.2: now also P4.2 (Pin_2); no longer P6.2 (Pin_2)
- net at P5.2 (Pin_2): now also C18.1, R8.2
- net at R29.2: now also L11.2, R30.2
- net at J9.1 (In): now also C30.2; no longer C21.2
- net at J4.1 (In): now also C19.1; no longer C51.1
- net at C51.2: now also C29.1, Q3.1 (B), R16.2
- net at J8.1 (In): now also C31.1; no longer C19.1
- net at J3.1 (In): now also C20.2
- net at C53.2: now also C33.1, Q5.1 (B), R23.2
- net at C54.1: now also R30.1
- net at R10.1: now also P6.2 (Pin_2), C27.1
- net at C53.1: now also R15.1
- net at J13.1 (In): now also C36.2
- net at J14.1 (In): now also C38.1
- net at C15.1, R42.1, U1.3 (RFIN): now also L12.1; no longer R19.1
- net at L11.1: now also Q6.3 (C), R31.1
- net at J5.1 (In): now also C21.2
- net at J7.1 (In): now also C29.2; no longer C20.2
- net at C58.2, R49.2, U1.4 (RFOUT): now also L26.1, R41.1
- net at R44.1: now also C63.1, L25.1, L26.2, R41.2
- net at P8.2 (Pin_2): now also C34.1, R14.1
- net at R10.2: now also R16.1, R18.1
- net at J10.1 (In): now also C32.1; no longer C22.1
- net at C54.2: now also C36.1, Q6.1 (B), R26.2
- net at J12.1 (In): now also C35.1
- new net: C30.1, C52.2, Q4.1 (B), R17.2
- new net: C37.1, P9.2 (Pin_2), R28.1
- new net: R14.2, R23.1, R24.1
- new net: C38.2, R31.2
- new net: Q4.3 (C), R13.2, R21.2, R22.1
- new net: C28.1, P7.2 (Pin_2), R12.1
- new net: Q5.3 (C), R15.2, R24.2, R25.1
- new net: Q3.3 (C), R11.2, R18.2, R20.1
- new net: R12.2, R17.1, R21.1
- new net: C35.2, R25.2
- new net: C63.2, R40.1
- new net: C32.2, R22.2
- new net: C31.2, R20.2
- new net: L12.2, R19.1
- new net: C51.1, R11.1
- new net: R26.1, R28.2, R29.1
- new net: C52.1, R13.1
Other:
- moved on the sheet: C15, C17, C18, C19, C20, C21, C22, C39, C45, C46, C59, J1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
