File: evaluation-boards/rf-amps/rf-amps.kicad_sch (KiCad schematic)
At the start: 103 parts, among them J1 CONN_COAXIAL, J10 CONN_COAXIAL, J11 CONN_COAXIAL, J12 CONN_COAXIAL, J13 CONN_COAXIAL, J14 CONN_COAXIAL, J2 CONN_COAXIAL, J3 CONN_COAXIAL, J4 CONN_COAXIAL, J5 CONN_COAXIAL, J6 CONN_COAXIAL, J7 CONN_COAXIAL, J8 CONN_COAXIAL, J9 CONN_COAXIAL, P1 Conn_01x02, P2 Conn_01x02, P3 CONN_01X03, P4 CONN_01X03, P5 CONN_01X03, P6 CONN_01X03, P7 CONN_01X03, P8 CONN_01X03, P9 CONN_01X03, Q1 BFR840, Q2 BFR840, Q3 BFP840ESD, Q4 BFP840ESD, Q5 BFP840ESD, Q6 BFP840ESD, U1 BGB741L7ESD

Commit message: Update rf-amps board
Parts:
- removed C11, C17, C18, C19, C20, C21, C22, C29, C30, C31, C32, C33, C35, C36, C38, C45, C46, C51, C52, C54, C57, C63: 1 uF, Capacitor_SMD:C_0201_0603Metric, symbol Device:C
- removed C15, C39: 220 nF, Capacitor_SMD:C_0201_0603Metric, symbol Device:C
- removed C27, C28, C34, C37: 1uF, Capacitor_SMD:C_0201_0603Metric, symbol Device:C
- removed C40: 0.3 pF, Capacitor_SMD:C_0201_0603Metric, symbol Device:C
- removed J10, J11, J12, J13, J14, J7, J8, J9: CONN_COAXIAL, sma-variants:SMA-EDGE-1.3mm-pad-1.05mm-gap-2.6mm-keepout, symbol Connector:Conn_Coaxial
- removed L10, L11, L14: 1.5 nH, Inductor_SMD:L_0201_0603Metric, symbol Device:L
- removed P6, P7, P8, P9: CONN_01X03, Connector_PinHeader_2.54mm:PinHeader_1x03_P2.54mm_Vertical, symbol Connector_Generic:Conn_01x03
- removed Q1, Q2: BFR840, eval:TSLP-3-9, symbol Transistor_BJT:Q_NPN_BCE
- removed Q3, Q4, Q5, Q6: BFP840ESD, eval:SOT-343-4-3, symbol eval:Q_NPN_BECE
- removed R10, R12, R14, R28: 75, Resistor_SMD:R_0201_0603Metric, symbol Device:R
- removed R11, R13, R15, R30, R4, R7: 240, Resistor_SMD:R_0201_0603Metric, symbol Device:R
- removed R16, R17, R23, R26: 27k, Resistor_SMD:R_0201_0603Metric, symbol Device:R
- removed R18, R21, R24, R29: 51, Resistor_SMD:R_0201_0603Metric, symbol Device:R
- removed R19: 180, Resistor_SMD:R_0201_0603Metric, symbol Device:R
- removed R20, R22, R25, R31: 15, Resistor_SMD:R_0201_0603Metric, symbol Device:R
- removed R27: 3.3k, Resistor_SMD:R_0201_0603Metric, symbol Device:R
- removed R3, R6: 33k, Resistor_SMD:R_0201_0603Metric, symbol Device:R
- removed R40, R41, R5, R8: 220, Resistor_SMD:R_0201_0603Metric, symbol Device:R
- removed R44: 6.8k, Resistor_SMD:R_0201_0603Metric, symbol Device:R
- removed R49: 3, Resistor_SMD:R_0201_0603Metric, symbol Device:R
- removed R52, R53: 1, Resistor_SMD:R_0201_0603Metric, symbol Device:R
- removed U1: BGB741L7ESD, rf-amps:TSLP-7-1, symbol gsg-symbols:BGB741L7ESD
- added C114, C139, C160, C161, C185, C195, C196, C197, C198, C205, C206, C50, C62, C78: 1 uF, Capacitor_SMD:C_0201_0603Metric, symbol Device:C
- added C187: 0.3pF, Capacitor_SMD:C_0201_0603Metric, symbol Device:C
- added L28: 2.4 nH, Inductor_SMD:L_0201_0603Metric, symbol Device:L
- added L5: 56 nH, Inductor_SMD:L_0201_0603Metric, symbol Device:L
- added Q11, Q14: Q_PMOS_GSD, eval:TSLP-3-9, symbol Transistor_FET:Q_PMOS_GSD
- added Q2: BFP840, eval:SOT-343-4-3, symbol eval:Q_NPN_BECE
- added Q8: BFR840, eval:TSLP-3-9, symbol Transistor_BJT:Q_NPN_BCE
- added R114, R140, R141, R146: 33k, Resistor_SMD:R_0201_0603Metric, symbol Device:R
- added R115, R116: 120, Resistor_SMD:R_0201_0603Metric, symbol Device:R
- added R117: 1, Resistor_SMD:R_0201_0603Metric, symbol Device:R
- added R123: 12k, Resistor_SMD:R_0201_0603Metric, symbol Device:R
- added R124: 180, Resistor_SMD:R_0201_0603Metric, symbol Device:R
- added R126: 300, Resistor_SMD:R_0201_0603Metric, symbol Device:R
- added R127: 3.3k, Resistor_SMD:R_0201_0603Metric, symbol Device:R
- added R128: 6.8k, Resistor_SMD:R_0201_0603Metric, symbol Device:R
- added R129, R131: 220, Resistor_SMD:R_0201_0603Metric, symbol Device:R
- added R132: 1k, Resistor_SMD:R_0201_0603Metric, symbol Device:R
- added R137: 100, Resistor_SMD:R_0201_0603Metric, symbol Device:R
- added R138: 51, Resistor_SMD:R_0201_0603Metric, symbol Device:R
- added R139: 10, Resistor_SMD:R_0201_0603Metric, symbol Device:R
- added R43: 3, Resistor_SMD:R_0201_0603Metric, symbol Device:R
- added U25: BGB741L7ESD, eval:TSLP-7-1, symbol eval:BGB741L7ESD
- C53, C58, C59: Manufacturer (none) -> Murata; Part Number (none) -> GRM033R61A105ME44D; Substitution (none) -> GRM033R61A105ME44*, GRM033R61C105ME15*, Samsung CL03A105MO3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
- J1, J2, J3, J4, J5, J6: footprint sma-variants:SMA-EDGE-1.3mm-pad-1.05mm-gap-2.6mm-keepout -> eval:SMA_MyAntenna_A-SMA-KE-16.5A_EdgeMount
- L12: value 8.2 nH -> 56 nH; Manufacturer (none) -> Murata; Part Number (none) -> LQP03TN56NJ02D; Substitution (none) -> LQP03TN56NH02D
- L25: value 100 uH -> 8.2 nH; footprint Inductor_SMD:L_0805_2012Metric -> Inductor_SMD:L_0201_0603Metric; Manufacturer (none) -> Murata; Part Number (none) -> LQP03TN8N2J02D; Substitution (none) -> LQP03TN8N2H02D
- L26: value 56 nH -> 100uH; footprint Inductor_SMD:L_0201_0603Metric -> eval:L_TDK_MLZ2012_h1.25mm; Manufacturer (none) -> TDK; Part Number (none) -> MLZ2012N101LT000; Substitution (none) -> MLZ2012N101LTD25
- R42: value 300 -> 220; Manufacturer (none) -> Yageo; Part Number (none) -> RC0201JR-07220RL; Substitution (none) -> any equivalent
Connections:
- net GND: now also C53.2, C114.2, C160.2, C161.2, C187.2, C196.2, C205.2, C206.2, Q2.2 (E), Q2.4 (C), Q8.3 (E), R131.1, R140.2, U25.7 (GND); no longer C59.1
- net at J2.1 (In): now also C187.1, C62.2
- net at J1.1 (In): now also C59.1
- net at P4.2 (Pin_2): now also Q14.1 (G), R146.2
- net at P5.2 (Pin_2): now also Q11.1 (G), R141.2
- net at J4.1 (In): now also C50.1
- net at R42.1: now also C53.1, Q14.2 (S); no longer L12.1
- net at C58.1: now also J3.1 (In); no longer R42.2
- net at L25.1: now also C59.2, R126.1, U25.3 (RFIN); no longer L26.2
- net at J5.1 (In): now also C195.2
- net at P3.2 (Pin_2): now also U25.5 (CTRL)
- net at C58.2: now also Q8.1 (B), R114.2, R116.2; no longer L26.1
- net at J6.1 (In): now also C198.1
- net at L12.2: now also C185.1, R129.1, R43.2, U25.4 (RFOUT)
- net VCC renamed VAA
- net VAA: now also L26.1, C160.1, C161.1, C205.1, C206.1, Q11.3 (D), Q14.3 (D), R127.1, R128.2, R141.1, R146.1, U25.1 (VCC); no longer C59.2, L25.2
- new net: C50.2, R117.1
- new net: C62.1, R43.1
- new net: L5.1, R114.1, R42.2
- new net: L5.2, Q8.2 (C), R115.1, R117.2
- new net: C139.2, R131.2
- new net: Q2.1 (B), R123.1, R132.1, R139.2, R140.1
- new net: C198.2, L28.1, Q2.3 (C)
- new net: R127.2, U25.6 (ADJ)
- new net: C78.1, R115.2
- new net: C139.1, L12.1, L26.2, R128.1, R129.2
- new net: L25.2, R124.1
- new net: C114.1, R124.2, U25.2 (BIAS)
- new net: C197.2, R132.2
- new net: C197.1, L28.2, R138.2
- new net: C196.1, Q11.2 (S), R137.1
- new net: C185.2, R126.2
- new net: R123.2, R137.2, R138.1
- new net: C195.1, R139.1
- new net: C78.2, R116.1
Other:
- moved on the sheet: J1, J2, J3, J4, J5, J6, P1, P2, P3, P4, P5
